File: DCOVoiceBoard/DCOVoiceBoard.kicad_pcb (KiCad board)
At the start: 4 copper layers, 150 x 50 mm, 162 parts, among them J101 ParentConn, Q201 BC857, Q202 BC857, Q301 BC858, Q302 BC858, Q401 BC858, Q402 BC857, Q403 BC847, Q404 BC857, Q405 BC847, Q406 BC858, U201 TL074, U202 TL074, U203 MCP4451-104E-ST, U204 TL074, U205 MCP4451-104E-ST, U206 TL072, U301 TL074, U302 TMUX4053, U303 LM13700, U304 MCP4018-103E/LT, U401 TMUX4053, U402 LM13700, U403 TL074, U404 TL072, U405 TL071

Commit message: motherboard hardware
Parts:
- removed C302, C303, C401, C402, C411, C412: 100n, Capacitor_SMD:C_0805_2012Metric
- removed R234, R235: 10k, PCM_Resistor_SMD_AKL:R_0805_2012Metric
- removed U302, U401: TMUX4053, Package_SO:TSSOP-16_4.4x5mm_P0.65mm
- removed U405: TL071, Package_SO:SOIC-8_3.9x4.9mm_P1.27mm
- added C101: 100n, Capacitor_SMD:C_0805_2012Metric, B.Cu at (71.8, 19.0)
- added C102: 100n, Capacitor_SMD:C_0805_2012Metric, B.Cu at (66.1, 8.63)
- added C103: 100n, Capacitor_SMD:C_0805_2012Metric, B.Cu at (71.6, 35.3)
- added C104: 100n, Capacitor_SMD:C_0805_2012Metric, B.Cu at (65.9, 25.5)
- added U101: TMUX4053, Package_SO:TSSOP-16_4.4x5mm_P0.65mm, B.Cu at (68.8, 30.4)
- added U102: TMUX4053, Package_SO:TSSOP-16_4.4x5mm_P0.65mm, B.Cu at (69.0, 13.9)
- C215, C216, C217, C218, R228, R229, R230, R231, R232, R233, R237, R238, R239, R240, R241, R242, U203, U204, U205: moved to B.Cu
- D301, D302: footprint LED_THT:LED_D3.0mm -> LED_SMD:LED_0805_2012Metric
- J101: value ParentConn -> VoiceHeader
- U303, U402: footprint PCM_Package_SO_AKL:SOIC-16_3.9x9.9mm_P1.27mm -> Package_SO:SOIC-16_3.9x9.9mm_P1.27mm
- U404: value TL072 -> TL074; footprint Package_SO:SOIC-8_3.9x4.9mm_P1.27mm -> Package_SO:SOIC-14_3.9x8.7mm_P1.27mm
- moved R404 146.5 mm to (125.2, 43.6)
- moved R402 145.9 mm to (115.5, 45.5)
- moved R401 145.4 mm to (115.0, 42.2), turned to 90 degrees
- moved R403 141.0 mm to (119.1, 38.8), turned to 180 degrees
- moved R425 133.4 mm to (104.0, 45.0), turned to -90 degrees
- moved R408 128.8 mm to (120.0, 35.7), turned to -90 degrees
- moved C405 128.3 mm to (119.2, 43.4)
- moved R412 127.3 mm to (124.4, 21.1)
- moved Q401 125.8 mm to (124.7, 39.3), turned to 90 degrees
- moved C404 123.9 mm to (114.9, 38.1), turned to 90 degrees
- moved C403 122.7 mm to (104.5, 40.9), turned to 180 degrees
- moved R413 122.5 mm to (124.4, 16.3), turned to 180 degrees
- moved R417 120.7 mm to (124.5, 6.55), turned to 180 degrees
- moved R429 119.5 mm to (98.0, 44.9), turned to 180 degrees
- moved R427 117.4 mm to (108.2, 28.9), turned to 90 degrees
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Connections:
- C403 pad 1: -12V -> +12V
- C404 pad 1: +12V -> -12V
- C405 pad 1: Net-(U405--) -> Net-(U404C--)
- J101 pad 10: HP_MODE -> PWM_1_CV
- J101 pad 11: LEVEL_1_CV -> FOLD_FIRST
- J101 pad 12: LEVEL_2_CV -> HP_MODE
- J101 pad 13: PWM_1_CV -> CUTOFF_CV
- J101 pad 14: PWM_2_CV -> FOLD_CV
- J101 pad 15: CUTOFF_CV -> VCA_CV
- J101 pad 16: FOLD_CV -> VCA_OUT
- J101 pad 17: VCA_CV -> SDA
- J101 pad 18: VCA_OUT -> SCL
- J101 pad 5: SDA -> CLK_2
- J101 pad 6: SCL -> CLK_1
- J101 pad 7: CLK_1 -> LEVEL_2_CV
- J101 pad 8: CLK_2 -> LEVEL_1_CV
- J101 pad 9: FOLD_FIRST -> PWM_2_CV
- R229 pad 1: Net-(U203A-P0W) -> Net-(U203D-P3W)
- R231 pad 1: Net-(U203D-P3W) -> Net-(U203A-P0W)
- R232 pad 2: Net-(U205D-P3B) -> Net-(U205A-P0B)
- R233 pad 2: Net-(U203D-P3B) -> Net-(U203A-P0B)
- R237 pad 1: Net-(U205A-P0W) -> Net-(U205D-P3W)
- R240 pad 1: Net-(U205D-P3W) -> Net-(U205A-P0W)
- R401 pad 1: Net-(U405--) -> Net-(U404C--)
- R402 pad 2: Net-(U405--) -> Net-(U404C--)
- R403 pad 2: Net-(U405--) -> Net-(U404C--)
- U203 pad 13: TRI1_FULL -> Net-(U203A-P0B)
- U203 pad 15: Net-(U203E-~{RESET}) -> +3.3V
- U203 pad 3: Net-(U203D-P3B) -> TRI1_FULL
- U204 pad 1: Net-(U205D-P3B) -> Net-(U205A-P0B)
- U204 pad 8: Net-(U203D-P3B) -> Net-(U203A-P0B)
- U205 pad 13: TRI2_FULL -> Net-(U205A-P0B)
- U205 pad 15: Net-(U205E-~{RESET}) -> +3.3V
- U205 pad 3: Net-(U205D-P3B) -> TRI2_FULL
- U404 pad 4: -12V -> +12V
- U404 pad 8: +12V -> Net-(Q401-B)
Routing:
- net -12V: track 0.00 -> 319.7 mm, vias 0 -> 14
- net GND: track 0.00 -> 161.4 mm, vias 0 -> 67
- net +3.3V: track 0.00 -> 156.4 mm, vias 0 -> 6
- net SAW2_FULL: track 0.00 -> 130.2 mm, vias 0 -> 5
- net SDA: track 0.00 -> 95.1 mm, vias 0 -> 4
- net SCL: track 0.00 -> 93.7 mm, vias 0 -> 3
- net PULSE2_FULL: track 0.00 -> 84.9 mm, vias 0 -> 1
- net FOLD_CV: track 0.00 -> 80.0 mm
- net CUTOFF_CV: track 0.00 -> 77.3 mm, vias 0 -> 1
- net SAW1_FULL: track 0.00 -> 75.0 mm, vias 0 -> 1
- net VCA_IN: track 0.00 -> 74.9 mm, vias 0 -> 3
- net PWM_2_CV: track 0.00 -> 68.9 mm, vias 0 -> 1
- net PWM_1_CV: track 0.00 -> 67.6 mm, vias 0 -> 1
- net HP_MODE: track 0.00 -> 66.8 mm, vias 0 -> 2
- net TRI2_FULL: track 0.00 -> 66.2 mm, vias 0 -> 1
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- added copper zone on In2.Cu, net +12V
- added copper zone on B.Cu, net GND
- added copper zone on F.Cu, net GND
- added copper zone on In1.Cu, net GND
Other:
- board size 150 x 50 mm -> 130 x 50 mm
- board text added: "+12V"
- board text added: "+3V3"
- board text added: "-12V"
- board text added: "AMP"
- board text added: "CLK1"
- board text added: "CLK2"
- board text added: "CUTOFF"
- board text added: "FLD_FRST"
- board text added: "FOLD"
- board text added: "GND"
- board text added: "HP_MODE"
- board text added: "LVL1"
- board text added: "LVL2"
- board text added: "PWM1"
- board text added: "PWM2"
- board text added: "SCL"
- board text added: "SDA"
- board text added: "VOICE OUT"
