File: DCOVoiceBoard/Filter.kicad_sch (KiCad schematic)
At the start: 35 parts, among them Q301 BC858, Q302 BC858, U301 TL074, U302 TMUX4053, U303 LM13700, U304 MCP4018-103E/LT

Commit message: voice board rough schematic
Parts:
- C301, C302, C303, C304, C305, C306, C307, C308, C309, C310, C311: footprint (none) -> Capacitor_SMD:C_0805_2012Metric
- D301, D302: footprint (none) -> LED_THT:LED_D3.0mm
- Q301, Q302: footprint Package_TO_SOT_SMD_AKL:SOT-23 -> PCM_Package_TO_SOT_SMD_AKL:SOT-23
- R301, R302, R303, R304, R305, R306, R307, R308, R309, R310, R311, R312, R313, R314, R315, R316: footprint (none) -> PCM_Resistor_SMD_AKL:R_0805_2012Metric
- U301: footprint (none) -> Package_SO:SOIC-14_3.9x8.7mm_P1.27mm
- U302: footprint (none) -> Package_SO:TSSOP-16_4.4x5mm_P0.65mm
- U303: footprint (none) -> PCM_Package_SO_AKL:SOIC-16_3.9x9.9mm_P1.27mm

Commit message: motherboard hardware
Parts:
- removed C302, C303: 100n, Capacitor_SMD:C_0805_2012Metric, symbol Device:C
- removed U302: TMUX4053, Package_SO:TSSOP-16_4.4x5mm_P0.65mm, symbol Analog_Switch:TMUX4053
- D301, D302: footprint LED_THT:LED_D3.0mm -> LED_SMD:LED_0805_2012Metric
- U303: footprint PCM_Package_SO_AKL:SOIC-16_3.9x9.9mm_P1.27mm -> Package_SO:SOIC-16_3.9x9.9mm_P1.27mm
Connections:
- no-connect marks 7 -> 6
Other:
- note removed: "Logic high on 'FOLD_FIRST' = route to the VCA, otherwise to the wave folder"
- note removed: "Logic high on HP_MODE = high pass mode"
- moved on the sheet: C301, C304, C305, C306, C307, C308, C309, C310, C311, D301, D302, Q301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
