File: PolySynthMotherboard/PolySynthMotherboard.kicad_pcb (KiCad board)
At the start: 4 copper layers, 542 parts, among them J201 SWD Header, J202 USB_C_Receptacle_USB2.0, J203 MIDI_In, J204 MIDI_Thru, J205 MIDI_Out, J206 Micro_SD_Card_Det2, J401 V1Header, J402 V2Header, J403 V3Header, J404 V4Header, J405 V5Header, J406 V6Header, J701 BATTERY, J702 POWER, J801 AUDIO_OUT, Q701 Q_PMOS_GSD, Q702 Q_PMOS_GSD, SW201 RST, SW202 BOOT, SW501 MM, SW502 MM, SW503 MM, SW504 MM, SW505 MM, SW506 MM, SW507 MM, SW508 MM, SW509 MM, SW510 MM, SW511 MM, SW512 MM, SW513 MM, SW514 MM, SW515 MM, SW516 MM, SW517 MM, SW518 MM, SW519 MM, SW520 MM, SW521 MM, SW522 MM, SW523 MM, SW524 MM, SW525 MM, SW526 MM, SW527 MM, SW528 MM, SW529 MM, SW530 MM, SW531 MM, SW532 MM, SW533 MM, SW534 MM, SW535 MM, SW536 MM, SW537 MM, SW538 MM, SW539 MM, SW540 MM, SW541 MM, SW542 MM, SW543 MM, SW544 MM, SW545 MM, SW546 MM, SW547 MM, SW548 MM, SW601 ENV1_B, SW602 ENV2_B, SW603 LFO1_B, SW604 LFO2_B, SW605 LFO3_B, SW606 MIX1_B, SW607 MIX2_B, SW608 MENU_B, SW609 FF_B, SW610 HP_B, SW611 HP_B, U201 STM32F411RETx, U202 74HC595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

Commit message: board layout
Parts:
- removed C320: 470n, Capacitor_SMD:C_0805_2012Metric
- added C383: 100n, Capacitor_SMD:C_0805_2012Metric, F.Cu at (120.7, -67.0)
- added C384: 100n, Capacitor_SMD:C_0805_2012Metric, F.Cu at (120.7, -64.0)
- added U303: TL072, Package_SO:SOIC-8_3.9x4.9mm_P1.27mm, F.Cu at (122.7, -71.8)
- C201, C202, C203, C204, C205, C206, C207, C208, C209, C210, C211, C212, C213, C214, C215, C216, C301, C304, C349, C350, C401, C602, C603, C604, C605, C606, C607, C608, C609, C611, C612, C613, C614, C615, C616, C617, C618, C620, C621, C702, C703, C711, D202, FB201, J201, J401, J402, J403, J404, J405, J406, R201, R202, R210, R401, R402, R403, R404, R405, R406, R407, R408, R409, R410, R411, R412, R413, R414, R415, R601, R602, R603, R604, R605, R606, R607, R608, R609, R610, R611, R612, R613, R614, R615, R616, R617, R618, R619, R620, R621, R622, R623, R624, R627, R628, SW201, SW202, U201, U202, U203, U301, U304, U306, U308, U309, U313, U317, U318, U401, Y201, Y202: moved to B.Cu
- D201: footprint Diode_THT:D_DO-35_SOD27_P7.62mm_Horizontal -> Diode_SMD:D_SOD-123
- D501, D502, D503, D504, D505, D506, D507, D508, D509, D510, D511, D512, D513, D514, D515, D516, D517, D518, D519, D520, D521, D522, D523, D524, D525, D526, D527, D528, D529, D530, D531, D532, D533, D534, D535, D536, D537, D538, D539, D540, D541, D542, D543, D544, D545, D546, D547, D548: footprint Diode_SMD:D_0805_2012Metric -> Diode_SMD:D_SOD-123; moved to B.Cu
- R304: value 10 -> 10k
- R810, R813: value 1k -> 470
- U205, U302, U305, U307, U310, U311, U312, U314, U315, U316, U319, U801: footprint PCM_Package_SO_AKL:SOIC-14_3.9x8.7mm_P1.27mm -> Package_SO:SOIC-14_3.9x8.7mm_P1.27mm
- U320: value TL074 -> TL072; footprint PCM_Package_SO_AKL:SOIC-14_3.9x8.7mm_P1.27mm -> Package_SO:SOIC-8_3.9x4.9mm_P1.27mm
- U701: footprint PCM_4ms_Package_SOIC:SOIC-8_5.28x4.9mm_Pitch1.27mm -> Package_SO:SOIC-8_3.9x4.9mm_P1.27mm
- moved RV801 499.0 mm to (282.6, 26.6), turned to 90 degrees
- moved J801 481.3 mm to (266.1, 2.29), turned to 90 degrees
- moved RE608 451.0 mm to (260.3, 52.6), turned to 90 degrees
- moved Y201 432.7 mm to (297.7, 71.5), turned to 135 degrees
- moved C618 430.2 mm to (268.5, 52.6)
- moved C707 429.3 mm to (313.2, 11.6), turned to -90 degrees
- moved RE607 427.9 mm to (234.4, 52.5), turned to 90 degrees
- moved C209 425.2 mm to (304.6, 85.2), turned to 90 degrees
- moved C216 425.2 mm to (310.5, 80.3), turned to -90 degrees
- moved C201 423.1 mm to (300.8, 63.4), turned to 45 degrees
- moved C205 422.4 mm to (302.4, 59.4), turned to -135 degrees
- moved RE606 422.3 mm to (213.0, 77.7), turned to 90 degrees
- moved C303 421.6 mm to (310.8, 116.9), turned to -90 degrees
- moved C706 421.1 mm to (305.0, 9.39), turned to 180 degrees
- moved RE605 420.7 mm to (212.9, 52.6), turned to 90 degrees
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Connections:
- C373 pad 1: Net-(U318-X5) -> Net-(U303B-+)
- C375 pad 1: Net-(U318-X4) -> Net-(U303A-+)
- J201 pad 1: GND -> +3.3V
- J201 pad 2: +3.3V -> TCK
- J201 pad 3: TCK -> GND
- J201 pad 5: SWO -> NRST
- J201 pad 6: NRST -> SWO
- R301 pad 1: Net-(U320D--) -> Net-(U320A--)
- R301 pad 2: Net-(U320C-+) -> Net-(U320B-+)
- R304 pad 2: Net-(U320D--) -> Net-(U320A--)
- R361 pad 1: Net-(U320C--) -> Net-(U320B--)
- R362 pad 2: Net-(U320C--) -> Net-(U320B--)
- U318 pad 1: Net-(U318-X4) -> Net-(U303A-+)
- U318 pad 5: Net-(U318-X5) -> Net-(U303B-+)
- U320 pad 1: VCA_V5 -> Net-(U320B-+)
- U320 pad 2: VCA_V5 -> Net-(U320A--)
- U320 pad 3: Net-(U318-X4) -> Net-(U301-VOUTG)
- U320 pad 4: +12V -> -12V
- U320 pad 5: Net-(U318-X5) -> Net-(U320B-+)
- U320 pad 6: VCA_V6 -> Net-(U320B--)
- U320 pad 7: VCA_V6 -> CUTOFF_DAC
- U320 pad 8: CUTOFF_DAC -> +12V
- U501 pad 1: MD_1 -> MD_8
- U501 pad 2: MD_2 -> MD_7
- U501 pad 3: MD_3 -> MD_6
- U501 pad 4: MD_4 -> MD_5
- U501 pad 5: MD_5 -> MD_4
- U501 pad 6: MD_6 -> MD_3
- U501 pad 7: MD_7 -> MD_2
- U501 pad 8: MD_8 -> MD_1
- U602 pad 1: ENCA_L -> ENCA_R
- U602 pad 2: ENCA_R -> ENCA_L
- U602 pad 21: ENV1_B -> MENU_B
- U602 pad 22: ENV2_B -> MIX2_B
- U602 pad 23: LFO1_B -> MIX1_B
- U602 pad 24: LFO2_B -> LFO3_B
- U602 pad 25: LFO3_B -> LFO2_B
- U602 pad 26: MIX1_B -> LFO1_B
- U602 pad 27: MIX2_B -> ENV2_B
- U602 pad 28: MENU_B -> ENV1_B
- U602 pad 3: ENCB_L -> ENCB_R
- U602 pad 4: ENCB_R -> ENCB_L
- U602 pad 5: ENCC_L -> ENCC_R
- U602 pad 6: ENCC_R -> ENCC_L
- U602 pad 7: ENCC_L -> ENCD_R
- U602 pad 8: ENCC_R -> ENCD_L

Commit message: new voice board proj
Parts:
- removed C309, C310: 100n, Capacitor_SMD:C_0805_2012Metric
- removed C313, C314, C315, C316, C317, C318, C319, C321, C322, C323, C324, C325, C330, C331, C332, C333, C334, C335, C336, C337, C338, C339, C340, C341, C342: 470n, Capacitor_SMD:C_0805_2012Metric
- removed U306: TMUX4051, Package_SO:TSSOP-16_4.4x5mm_P0.65mm
- C349, C350, D202, U304, U308, U309, U313, U317, U318: moved to F.Cu
- C383, C384, C801, C802, C803, R301, R304, R361, R362, R801, R802, R803, R804, R805, R806, R807, R808, R809, R810, R811, R812, R813, U320, U801: moved to B.Cu
- J202: value USB_C_Receptacle_USB2.0 -> USB_C_Leceptacle_USB2.0
- RE606: value ENC_RES -> ENC_LES
- moved R808 498.0 mm to (270.6, 13.0), turned to 180 degrees
- moved C801 496.2 mm to (262.7, 16.1)
- moved R810 492.0 mm to (261.5, 7.29), turned to 90 degrees
- moved R813 489.7 mm to (265.2, 7.29), turned to 90 degrees
- moved C803 489.5 mm to (251.2, 4.79), turned to 90 degrees
- moved C802 485.6 mm to (251.2, 16.3), turned to -90 degrees
- moved C373 482.2 mm to (439.9, 229.0)
- moved C375 481.4 mm to (435.7, 237.6), turned to -90 degrees
- moved R807 480.8 mm to (254.4, 16.1)
- moved R812 480.2 mm to (255.4, 4.00)
- moved R804 475.7 mm to (244.8, 23.1), turned to 90 degrees
- moved R809 474.8 mm to (246.9, 16.7), turned to 180 degrees
- moved R805 472.7 mm to (241.0, 23.1), turned to 90 degrees
- moved U801 471.8 mm to (251.2, 10.5), turned to 90 degrees
- moved C374 470.5 mm to (431.4, 223.8), turned to -90 degrees
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Connections:
- net AUDIO_OUT_R renamed AUDIO_OUT_L
- net BATT_REF renamed BATT_LEF
- net DISP_RST renamed DISP_LST
- net I2C_MUX_RST renamed I2C_MUX_LST
- net MIDI_RX renamed MIDI_LX
- C602 pad 1: ENCA_R -> ENCA_L
- C603 pad 1: ENCA_L -> ENCA_R
- C604 pad 1: ENCB_R -> ENCB_L
- C605 pad 1: ENCB_L -> ENCB_R
- C606 pad 1: ENCC_R -> ENCC_L
- C607 pad 1: ENCC_L -> ENCC_R
- C608 pad 1: ENCD_R -> ENCD_L
- C609 pad 1: ENCD_L -> ENCD_R
- C611 pad 1: ENCCF_R -> ENCCF_L
- C612 pad 1: ENCCF_L -> ENCCF_R
- C613 pad 1: ENCRES_R -> ENCRES_L
- C614 pad 1: ENCRES_L -> ENCRES_R
- C615 pad 1: ENCPWM_R -> ENCPWM_L
- C616 pad 1: ENCPWM_L -> ENCPWM_R
- C617 pad 1: ENCFOLD_R -> ENCFOLD_L
- C618 pad 1: ENCFOLD_L -> ENCFOLD_R
- C620 pad 1: ENCDEPTH_R -> ENCDEPTH_L
- C621 pad 1: ENCDEPTH_L -> ENCDEPTH_R
- J401 pad 3: +3.3VA -> +3.3V
- J402 pad 3: +3.3VA -> +3.3V
- J403 pad 3: +3.3VA -> +3.3V
- J404 pad 3: +3.3VA -> +3.3V
- J405 pad 3: +3.3VA -> +3.3V
- J406 pad 3: +3.3VA -> +3.3V
- R601 pad 2: ENCA_R -> ENCA_L
- R602 pad 2: ENCA_L -> ENCA_R
- R605 pad 2: ENCB_R -> ENCB_L
- R606 pad 2: ENCB_L -> ENCB_R
- R608 pad 2: ENCC_R -> ENCC_L
- R609 pad 2: ENCC_L -> ENCC_R
- R611 pad 2: ENCD_R -> ENCD_L
- R612 pad 2: ENCD_L -> ENCD_R
- R617 pad 2: ENCCF_R -> ENCCF_L
- R618 pad 2: ENCCF_L -> ENCCF_R
- R619 pad 2: ENCRES_R -> ENCRES_L
- R620 pad 2: ENCRES_L -> ENCRES_R
- R621 pad 2: ENCPWM_R -> ENCPWM_L
- R622 pad 2: ENCPWM_L -> ENCPWM_R
- R623 pad 2: ENCFOLD_R -> ENCFOLD_L
- R624 pad 2: ENCFOLD_L -> ENCFOLD_R
- R627 pad 2: ENCDEPTH_R -> ENCDEPTH_L
- R628 pad 2: ENCDEPTH_L -> ENCDEPTH_R
- RE601 pad A: ENCA_R -> ENCA_L
- RE601 pad B: ENCA_L -> ENCA_R
- RE602 pad A: ENCB_R -> ENCB_L
- RE602 pad B: ENCB_L -> ENCB_R
- RE603 pad A: ENCC_R -> ENCC_L
- RE603 pad B: ENCC_L -> ENCC_R
- RE604 pad A: ENCD_R -> ENCD_L
- RE604 pad B: ENCD_L -> ENCD_R
- RE605 pad A: ENCCF_R -> ENCCF_L
- RE605 pad B: ENCCF_L -> ENCCF_R
- RE606 pad A: ENCRES_R -> ENCRES_L
- RE606 pad B: ENCRES_L -> ENCRES_R
- RE607 pad A: ENCPWM_R -> ENCPWM_L
- RE607 pad B: ENCPWM_L -> ENCPWM_R
- RE608 pad A: ENCFOLD_R -> ENCFOLD_L
- RE608 pad B: ENCFOLD_L -> ENCFOLD_R
- RE609 pad A: ENCDEPTH_R -> ENCDEPTH_L
- RE609 pad B: ENCDEPTH_L -> ENCDEPTH_R
- U301 pad 8: +3.3VA -> +3.3V
- U301 pad 9: +3.3VA -> +3.3V
- U602 pad 1: ENCA_R -> ENCA_L
- U602 pad 2: ENCA_L -> ENCA_R
- U602 pad 3: ENCB_R -> ENCB_L
- U602 pad 4: ENCB_L -> ENCB_R
- U602 pad 5: ENCC_R -> ENCC_L
- U602 pad 6: ENCC_L -> ENCC_R
- U602 pad 7: ENCD_R -> ENCD_L
- U602 pad 8: ENCD_L -> ENCD_R
- U603 pad 21: ENCCF_L -> ENCFOLD_R
- U603 pad 22: ENCCF_R -> ENCFOLD_L
- U603 pad 23: ENCRES_L -> ENCPWM_R
- U603 pad 24: ENCRES_R -> ENCPWM_L
- U603 pad 25: ENCPWM_L -> ENCRES_R
- U603 pad 26: ENCPWM_R -> ENCRES_L
- U603 pad 27: ENCFOLD_L -> ENCCF_R
- U603 pad 28: ENCFOLD_R -> ENCCF_L
- U603 pad 7: ENCDEPTH_L -> ENCDEPTH_R
- U603 pad 8: ENCDEPTH_R -> ENCDEPTH_L
Routing:
- added copper zone on In1.Cu, net +3.3V
- added copper zone on In2.Cu, net GND
- added copper zone on F.Cu, net GNDPWR

Commit message: op-amp layout improved
Parts:
- removed J401: V1Header, Connector_PinSocket_2.54mm:PinSocket_1x18_P2.54mm_Vertical
- removed J402: V2Header, Connector_PinSocket_2.54mm:PinSocket_1x18_P2.54mm_Vertical
- removed J403: V3Header, Connector_PinSocket_2.54mm:PinSocket_1x18_P2.54mm_Vertical
- removed J404: V4Header, Connector_PinSocket_2.54mm:PinSocket_1x18_P2.54mm_Vertical
- removed J405: V5Header, Connector_PinSocket_2.54mm:PinSocket_1x18_P2.54mm_Vertical
- removed J406: V6Header, Connector_PinSocket_2.54mm:PinSocket_1x18_P2.54mm_Vertical
- added C309: 100n, Capacitor_SMD:C_0805_2012Metric, F.Cu at (381.9, 141.6)
- added C310: 100n, Capacitor_SMD:C_0805_2012Metric, F.Cu at (372.2, 135.9)
- added C313: 470n, Capacitor_SMD:C_0805_2012Metric, F.Cu at (445.4, 137.3)
- added C314: 470n, Capacitor_SMD:C_0805_2012Metric, F.Cu at (445.4, 140.3)
- added C315: 470n, Capacitor_SMD:C_0805_2012Metric, F.Cu at (445.4, 143.3)
- added C316: 470n, Capacitor_SMD:C_0805_2012Metric, F.Cu at (445.4, 146.3)
- added C317: 470n, Capacitor_SMD:C_0805_2012Metric, F.Cu at (445.4, 149.3)
- added C318: 470n, Capacitor_SMD:C_0805_2012Metric, F.Cu at (449.8, 131.3)
- added C319: 470n, Capacitor_SMD:C_0805_2012Metric, F.Cu at (449.8, 134.3)
- added C321: 470n, Capacitor_SMD:C_0805_2012Metric, F.Cu at (449.8, 137.3)
- added C322: 470n, Capacitor_SMD:C_0805_2012Metric, F.Cu at (449.8, 140.3)
- added C323: 470n, Capacitor_SMD:C_0805_2012Metric, F.Cu at (449.8, 143.3)
- added C324: 470n, Capacitor_SMD:C_0805_2012Metric, F.Cu at (449.8, 146.3)
- added C325: 470n, Capacitor_SMD:C_0805_2012Metric, F.Cu at (449.8, 149.3)
- added C330: 470n, Capacitor_SMD:C_0805_2012Metric, F.Cu at (454.2, 131.3)
- added C331: 470n, Capacitor_SMD:C_0805_2012Metric, F.Cu at (454.2, 134.3)
- added C332: 470n, Capacitor_SMD:C_0805_2012Metric, F.Cu at (454.2, 137.3)
- added C333: 470n, Capacitor_SMD:C_0805_2012Metric, F.Cu at (454.2, 140.3)
- added C334: 470n, Capacitor_SMD:C_0805_2012Metric, F.Cu at (454.2, 143.3)
- added C335: 470n, Capacitor_SMD:C_0805_2012Metric, F.Cu at (454.2, 146.3)
- added C336: 470n, Capacitor_SMD:C_0805_2012Metric, F.Cu at (454.2, 149.3)
- added C337: 470n, Capacitor_SMD:C_0805_2012Metric, F.Cu at (458.7, 131.3)
- added C338: 470n, Capacitor_SMD:C_0805_2012Metric, F.Cu at (458.7, 134.3)
- added C339: 470n, Capacitor_SMD:C_0805_2012Metric, F.Cu at (458.7, 137.3)
- added C340: 470n, Capacitor_SMD:C_0805_2012Metric, F.Cu at (458.7, 140.3)
- added C342: 470n, Capacitor_SMD:C_0805_2012Metric, F.Cu at (458.7, 143.3)
- added U306: TMUX4051, Package_SO:TSSOP-16_4.4x5mm_P0.65mm, F.Cu at (377.1, 138.8)
- added U402: Voice1, Connector_PinHeader_2.54mm:PinHeader_2x09_P2.54mm_Vertical, B.Cu at (248.2, 130.6)
- added U403: Voice2, Connector_PinHeader_2.54mm:PinHeader_2x09_P2.54mm_Vertical, B.Cu at (168.9, 136.2)
- added U404: Voice3, Connector_PinHeader_2.54mm:PinHeader_2x09_P2.54mm_Vertical, B.Cu at (248.2, 116.2)
- added U405: Voice4, Connector_PinHeader_2.54mm:PinHeader_2x09_P2.54mm_Vertical, B.Cu at (168.9, 121.8)
- added U406: Voice5, Connector_PinHeader_2.54mm:PinHeader_2x09_P2.54mm_Vertical, B.Cu at (248.2, 101.8)
- added U407: Voice6, Connector_PinHeader_2.54mm:PinHeader_2x09_P2.54mm_Vertical, B.Cu at (168.9, 107.4)
- moved C303 213.6 mm to (183.2, 139.8)
- moved C302 213.6 mm to (183.2, 127.7)
- moved R302 213.6 mm to (177.4, 139.8)
- moved R303 213.6 mm to (179.7, 139.8)
- moved R305 213.6 mm to (189.1, 127.7)
- moved R307 213.6 mm to (189.1, 139.8)
- moved R309 213.6 mm to (179.7, 127.6)
- moved U302 213.6 mm to (182.7, 133.5)
- moved R308 213.6 mm to (186.8, 139.8)
- moved R310 213.6 mm to (177.4, 127.6)
- moved R306 213.6 mm to (186.8, 127.7)
- moved R314 213.0 mm to (176.8, 102.9), turned to -90 degrees
- moved R313 209.0 mm to (179.0, 102.9), turned to 90 degrees
- moved R324 205.3 mm to (176.8, 114.8), turned to 90 degrees
- moved C307 202.1 mm to (182.7, 102.8), turned to 90 degrees
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Connections:
- net I2C_MUX_LST renamed I2C_MUX_RST
- R302 pad 2: LVL1_V1 -> LVL1_V2
- R308 pad 2: LVL1_V2 -> LVL1_V1
- R317 pad 2: LVL2_V5 -> LVL2_V3
- R318 pad 2: LVL2_V3 -> LVL2_V2
- R321 pad 2: LVL2_V6 -> LVL2_V4
- R322 pad 2: LVL2_V4 -> LVL2_V1
- R324 pad 2: LVL2_V1 -> LVL2_V6
- R326 pad 2: LVL2_V2 -> LVL2_V5
- R333 pad 2: PWM2_V1 -> PWM2_V6
- R334 pad 2: PWM2_V5 -> PWM2_V3
- R335 pad 2: PWM2_V3 -> PWM2_V2
- R338 pad 2: PWM1_V1 -> PWM1_V2
- R345 pad 2: PWM2_V6 -> PWM2_V4
- R346 pad 2: PWM2_V4 -> PWM2_V1
- R349 pad 2: PWM2_V2 -> PWM2_V5
- R350 pad 2: PWM1_V2 -> PWM1_V1
- R406 pad 2: SDA_V2 -> SCL_V2
- R407 pad 2: SCL_V2 -> SDA_V2
- R408 pad 2: SDA_V3 -> SCL_V3
- R409 pad 2: SCL_V3 -> SDA_V3
- R410 pad 2: SDA_V4 -> SCL_V4
- R411 pad 2: SCL_V4 -> SDA_V4
- R412 pad 2: SDA_V5 -> SCL_V5
- R413 pad 2: SCL_V5 -> SDA_V5
- R414 pad 2: SDA_V6 -> SCL_V6
- R415 pad 2: SCL_V6 -> SDA_V6
- R706 pad 2: BATT_LEF -> BATT_REF
- R707 pad 1: BATT_LEF -> BATT_REF
- U201 pad 10: unconnected-(U201-PC2-Pad10) -> FOLD_FIRST
- U201 pad 26: unconnected-(U201-PB0-Pad26) -> BATT_REF
- U201 pad 9: BATT_LEF -> HP_MODE
- U302 pad 1: LVL1_V1 -> LVL1_V2
- U302 pad 7: LVL1_V2 -> LVL1_V1
- U304 pad 13: Net-(U302A-+) -> Net-(U302B-+)
- U304 pad 14: Net-(U302B-+) -> Net-(U302A-+)
- U305 pad 14: LVL2_V2 -> LVL2_V5
- U305 pad 8: LVL2_V1 -> LVL2_V6
- U307 pad 1: LVL2_V3 -> LVL2_V2
- U307 pad 14: LVL2_V6 -> LVL2_V4
- U307 pad 7: LVL2_V4 -> LVL2_V1
- U307 pad 8: LVL2_V5 -> LVL2_V3
- U310 pad 10: Net-(U308-X0) -> Net-(U308-X5)
- U310 pad 12: Net-(U308-X1) -> Net-(U308-X4)
- U310 pad 14: PWM2_V2 -> PWM2_V5
- U310 pad 8: PWM2_V1 -> PWM2_V6
- U311 pad 1: PWM2_V3 -> PWM2_V2
- U311 pad 10: Net-(U308-X4) -> Net-(U308-X2)
- U311 pad 12: Net-(U308-X5) -> Net-(U308-X3)
- U311 pad 14: PWM2_V6 -> PWM2_V4
- U311 pad 3: Net-(U308-X2) -> Net-(U308-X1)
- U311 pad 5: Net-(U308-X3) -> Net-(U308-X0)
- U311 pad 7: PWM2_V4 -> PWM2_V1
- U311 pad 8: PWM2_V5 -> PWM2_V3
- U312 pad 1: PWM1_V1 -> PWM1_V2
- U312 pad 3: Net-(U309-X0) -> Net-(U309-X1)
- U312 pad 5: Net-(U309-X1) -> Net-(U309-X0)
- U312 pad 7: PWM1_V2 -> PWM1_V1

Commit message: power supply tweaks
Parts:
- removed D501, D502, D503, D504, D505, D506, D507, D508, D509, D510, D511, D512, D513, D514, D515, D516, D517, D518, D519, D520, D521, D522, D523, D524, D525, D526, D527, D528, D529, D530, D531, D532, D533, D534, D535, D536, D537, D538, D539, D540, D541, D542, D543, D544, D545, D546, D547, D548: 1N4148, Diode_SMD:D_SOD-123
- removed SW515, SW516, SW517, SW518, SW519, SW520, SW521, SW522, SW523, SW524, SW525, SW526, SW527, SW528, SW529, SW530, SW531, SW532, SW533, SW534, SW535, SW536, SW537, SW538, SW539, SW540, SW541, SW542, SW543, SW544, SW545, SW546, SW547, SW548: MM, Button_Switch_THT:SW_PUSH_6mm
- added R509: 47k, PCM_Resistor_SMD_AKL:R_0805_2012Metric, F.Cu at (8.31, 96.9)
- added R510: 47k, PCM_Resistor_SMD_AKL:R_0805_2012Metric, F.Cu at (8.08, 83.7)
- added R511: 47k, PCM_Resistor_SMD_AKL:R_0805_2012Metric, F.Cu at (8.07, 71.0)
- added R512: 47k, PCM_Resistor_SMD_AKL:R_0805_2012Metric, F.Cu at (8.08, 58.1)
- added R513: 47k, PCM_Resistor_SMD_AKL:R_0805_2012Metric, F.Cu at (8.06, 45.6)
- added R514: 47k, PCM_Resistor_SMD_AKL:R_0805_2012Metric, F.Cu at (7.97, 32.7)
- C305, C306, C309, C310, C313, C314, C315, C316, C317, C318, C319, C321, C322, C323, C324, C325, C326, C327, C328, C329, C330, C331, C332, C333, C334, C335, C336, C337, C338, C339, C340, C342, C349, C350, C358, C359, C371, C372, C501, U304, U306, U308, U309, U313, U317, U318, U501: moved to B.Cu
- SW501: value MM -> MD1
- SW502: value MM -> MD2
- SW503: value MM -> MD3
- SW504: value MM -> MD4
- SW505: value MM -> MD5
- SW506: value MM -> MD6
- SW507: value MM -> MD7
- SW508: value MM -> MD8
- SW509: value MM -> MS1
- SW510: value MM -> MS2
- SW511: value MM -> MS3
- SW512: value MM -> MS4
- SW513: value MM -> MS5
- SW514: value MM -> MS6
- moved C317 434.2 mm to (19.9, 62.6), turned to 90 degrees
- moved C315 432.4 mm to (17.8, 78.5), turned to -90 degrees
- moved C318 431.8 mm to (23.5, 62.6), turned to 90 degrees
- moved C313 430.0 mm to (19.9, 74.9), turned to -90 degrees
- moved C314 428.5 mm to (21.4, 78.5), turned to -90 degrees
- moved C316 427.9 mm to (23.5, 74.9), turned to -90 degrees
- moved C324 424.0 mm to (34.3, 61.6), turned to 90 degrees
- moved C322 423.2 mm to (31.7, 74.9), turned to -90 degrees
- moved C325 421.4 mm to (37.6, 61.6), turned to 90 degrees
- moved C321 420.3 mm to (33.6, 78.6), turned to -90 degrees
- moved C319 418.3 mm to (35.8, 74.9), turned to -90 degrees
- moved C339 417.9 mm to (45.4, 75.0), turned to -90 degrees
- moved C323 417.6 mm to (37.2, 78.6), turned to -90 degrees
- moved C342 417.1 mm to (46.6, 78.7), turned to -90 degrees
- moved C336 416.8 mm to (46.6, 62.6), turned to 90 degrees
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Connections:
- C353 pad 1: Net-(U313-X2) -> Net-(U313-X4)
- C355 pad 1: Net-(U313-X4) -> Net-(U313-X2)
- C357 pad 1: Net-(U315C-+) -> Net-(U314D-+)
- C361 pad 1: Net-(U316A-+) -> Net-(U317-X2)
- C362 pad 1: Net-(U316B-+) -> Net-(U316A-+)
- C369 pad 1: Net-(U316C-+) -> Net-(U317-X4)
- C370 pad 1: Net-(U316D-+) -> Net-(U316B-+)
- C377 pad 1: Net-(U318-X1) -> Net-(U316C-+)
- C378 pad 1: Net-(U318-X3) -> Net-(U316D-+)
- R334 pad 2: PWM2_V3 -> PWM2_V4
- R335 pad 2: PWM2_V2 -> PWM2_V1
- R345 pad 2: PWM2_V4 -> PWM2_V3
- R346 pad 2: PWM2_V1 -> PWM2_V2
- SW501 pad 1: Net-(D501-A) -> GND
- SW502 pad 1: Net-(D502-A) -> GND
- SW503 pad 1: Net-(D503-A) -> GND
- SW504 pad 1: Net-(D504-A) -> GND
- SW505 pad 1: Net-(D505-A) -> GND
- SW506 pad 1: Net-(D506-A) -> GND
- SW507 pad 1: Net-(D507-A) -> GND
- SW508 pad 1: Net-(D508-A) -> GND
- SW509 pad 1: Net-(D509-A) -> GND
- SW509 pad 2: MD_1 -> MS_1
- SW510 pad 1: Net-(D510-A) -> GND
- SW510 pad 2: MD_2 -> MS_2
- SW511 pad 1: Net-(D511-A) -> GND
- SW511 pad 2: MD_3 -> MS_3
- SW512 pad 1: Net-(D512-A) -> GND
- SW512 pad 2: MD_4 -> MS_4
- SW513 pad 1: Net-(D513-A) -> GND
- SW513 pad 2: MD_5 -> MS_5
- SW514 pad 1: Net-(D514-A) -> GND
- SW514 pad 2: MD_6 -> MS_6
- U201 pad 14: unconnected-(U201-PA0-Pad14) -> BATT_REF
- U201 pad 26: BATT_REF -> DAC_INH
- U304 pad 6: GND -> DAC_INH
- U306 pad 6: GND -> DAC_INH
- U308 pad 6: GND -> DAC_INH
- U309 pad 6: GND -> DAC_INH
- U311 pad 1: PWM2_V2 -> PWM2_V1
- U311 pad 10: Net-(U308-X2) -> Net-(U308-X3)
- U311 pad 12: Net-(U308-X3) -> Net-(U308-X2)
- U311 pad 14: PWM2_V4 -> PWM2_V3
- U311 pad 3: Net-(U308-X1) -> Net-(U308-X0)
- U311 pad 5: Net-(U308-X0) -> Net-(U308-X1)
- U311 pad 7: PWM2_V1 -> PWM2_V2
- U311 pad 8: PWM2_V3 -> PWM2_V4
- U313 pad 6: GND -> DAC_INH
- U314 pad 12: Net-(U313-X3) -> Net-(U314D-+)
- U314 pad 13: FOLD_V4 -> CUTOFF_V1
- U314 pad 14: FOLD_V4 -> CUTOFF_V1
- U314 pad 5: Net-(U313-X1) -> Net-(U313-X4)
- U314 pad 6: FOLD_V2 -> FOLD_V5
- U314 pad 7: FOLD_V2 -> FOLD_V5
- U315 pad 1: FOLD_V5 -> FOLD_V2
- U315 pad 10: Net-(U315C-+) -> Net-(U313-X5)
- U315 pad 2: FOLD_V5 -> FOLD_V2
- U315 pad 3: Net-(U313-X4) -> Net-(U313-X1)
- U315 pad 5: Net-(U313-X5) -> Net-(U313-X3)
- U315 pad 6: FOLD_V6 -> FOLD_V4
- U315 pad 7: FOLD_V6 -> FOLD_V4
- U315 pad 8: CUTOFF_V1 -> FOLD_V6
- U315 pad 9: CUTOFF_V1 -> FOLD_V6
- U316 pad 1: CUTOFF_V3 -> CUTOFF_V4
- U316 pad 13: CUTOFF_V6 -> VCA_V4
- U316 pad 14: CUTOFF_V6 -> VCA_V4
- U316 pad 2: CUTOFF_V3 -> CUTOFF_V4
- U316 pad 6: CUTOFF_V4 -> CUTOFF_V6
- U316 pad 7: CUTOFF_V4 -> CUTOFF_V6
- U316 pad 8: CUTOFF_V5 -> VCA_V2
- U316 pad 9: CUTOFF_V5 -> VCA_V2
- U317 pad 1: Net-(U316C-+) -> Net-(U317-X4)
- U317 pad 12: Net-(U316B-+) -> Net-(U316A-+)
- U317 pad 13: Net-(U315C-+) -> Net-(U314D-+)
- U317 pad 15: Net-(U316A-+) -> Net-(U317-X2)
- U317 pad 5: Net-(U316D-+) -> Net-(U316B-+)
- U317 pad 6: GND -> DAC_INH
- U318 pad 12: Net-(U318-X3) -> Net-(U316D-+)
- U318 pad 14: Net-(U318-X1) -> Net-(U316C-+)
- U318 pad 6: GND -> DAC_INH
- U319 pad 1: VCA_V1 -> CUTOFF_V3
- U319 pad 10: Net-(U318-X2) -> Net-(U318-X0)
- U319 pad 12: Net-(U318-X3) -> Net-(U318-X2)
- U319 pad 13: VCA_V4 -> VCA_V3
- U319 pad 14: VCA_V4 -> VCA_V3
- U319 pad 2: VCA_V1 -> CUTOFF_V3
- U319 pad 3: Net-(U318-X0) -> Net-(U317-X2)
- U319 pad 5: Net-(U318-X1) -> Net-(U317-X4)
- U319 pad 6: VCA_V2 -> CUTOFF_V5
- U319 pad 7: VCA_V2 -> CUTOFF_V5
- U319 pad 8: VCA_V3 -> VCA_V1
- U319 pad 9: VCA_V3 -> VCA_V1
Routing:
- net +12V: track 0.00 -> 279.8 mm
- net -12V: track 0.00 -> 235.4 mm
- net USB_D-: track 0.00 -> 60.7 mm, vias 0 -> 1
- net USB_D+: track 0.00 -> 57.5 mm, vias 0 -> 1
- net GND: track 0.00 -> 47.0 mm, vias 0 -> 20
- net SWO: track 0.00 -> 39.5 mm
- net VDD: track 0.00 -> 36.3 mm
- net BATT+: track 0.00 -> 34.5 mm, vias 0 -> 1
- net TMS: track 0.00 -> 33.8 mm
- net VCC: track 0.00 -> 33.6 mm, vias 0 -> 2
- net +3.3V: track 0.00 -> 28.5 mm, vias 0 -> 6
- net TCK: track 0.00 -> 27.0 mm
- net SCL_V2: track 0.00 -> 20.1 mm
- net SDA_V2: track 0.00 -> 18.8 mm
- net SW_P: track 0.00 -> 15.2 mm
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