File: PolySynthMotherboard/PolySynthMotherboard.kicad_pcb (KiCad board)
At the start: 4 copper layers, 467 parts, among them J201 SWD Header, J202 USB_C_Leceptacle_USB2.0, J203 MIDI_In, J204 MIDI_Thru, J205 MIDI_Out, J206 Micro_SD_Card_Det2, J701 BATTERY, J702 POWER, J801 AUDIO_OUT, Q701 Q_PMOS_GSD, Q702 Q_PMOS_GSD, SW201 RST, SW202 BOOT, SW501 MD1, SW502 MD2, SW503 MD3, SW504 MD4, SW505 MD5, SW506 MD6, SW507 MD7, SW508 MD8, SW509 MS1, SW510 MS2, SW511 MS3, SW512 MS4, SW513 MS5, SW514 MS6, SW601 ENV1_B, SW602 ENV2_B, SW603 LFO1_B, SW604 LFO2_B, SW605 LFO3_B, SW606 MIX1_B, SW607 MIX2_B, SW608 MENU_B, SW609 FF_B, SW610 HP_B, SW611 HP_B, U201 STM32F411RETx, U202 74HC595, U203 74HC595, U204 4N35, U205 74HC04, U301 DAC7578xPW, U302 TL074, U303 TL072, U304 TMUX4051, U305 TL074, U306 TMUX4051, U307 TL074, U308 TMUX4051, U309 TMUX4051, U310 TL074, U311 TL074, U312 TL074, U313 TMUX4051, U314 TL074, U315 TL074, U316 TL074, U317 TMUX4051, U318 TMUX4051, U319 TL074, U320 TL072, U401 TCA9548APWR, U402 Voice1, U403 Voice2, U404 Voice3, U405 Voice4, U406 Voice5, U407 Voice6, U501 MCP23S17_SS, U601 ILI9341, U602 MCP23S17_SS, U603 MCP23S17_SS, U701 CS5173, U702 TC7662Bx0A, U703 MAX1898, U704 TPS61200DRC, U705 TC7662Bx0A, U801 TL074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

Commit message: fixed git maybe
Parts:
- removed NT701, NT702: NetTie_2, NetTie:NetTie-2_SMD_Pad0.5mm
- removed R711: 1M, PCM_Resistor_SMD_AKL:R_0805_2012Metric
- removed R712: 180k, PCM_Resistor_SMD_AKL:R_0805_2012Metric
- removed TP704: +3V3, TestPoint:TestPoint_Pad_D1.0mm_Value
- removed TP705: VCC, TestPoint:TestPoint_Pad_D1.0mm_Value
- added C625: 10n, Capacitor_SMD:C_0805_2012Metric, F.Cu at (361.2, 65.1)
- added C626: 10n, Capacitor_SMD:C_0805_2012Metric, F.Cu at (361.2, 68.2)
- added C715: 1u, Capacitor_SMD:C_0805_2012Metric, F.Cu at (342.6, 73.2)
- added C716: 100n, Capacitor_SMD:C_0805_2012Metric, F.Cu at (342.6, 76.2)
- added C717: 1u, Capacitor_SMD:C_0805_2012Metric, F.Cu at (342.6, 79.2)
- added C718: 100n, Capacitor_SMD:C_0805_2012Metric, F.Cu at (342.6, 82.2)
- added C719: 22u, Capacitor_SMD:C_0805_2012Metric, F.Cu at (359.6, 125.0)
- added C720: 100n, Capacitor_SMD:C_0805_2012Metric, F.Cu at (359.6, 128.0)
- added D705: PMEG3030, PCM_Diode_SMD_AKL:D_SOD-123, F.Cu at (352.4, 81.3)
- added D706: PMEG3030, PCM_Diode_SMD_AKL:D_SOD-123, F.Cu at (352.4, 85.4)
- added JP703: POS_CM, Jumper:SolderJumper-2_Open_TrianglePad_0805, F.Cu at (342.6, 85.3)
- added JP704: NEG_CM, Jumper:SolderJumper-2_Open_TrianglePad_0805, F.Cu at (342.6, 88.6)
- added JP705: DIG_CM, Jumper:SolderJumper-2_Open_TrianglePad_0805, F.Cu at (367.6, 118.6)
- added Q703: TD6790, PCM_4ms_Package_SOIC:SM-8, F.Cu at (350.5, 75.5)
- added Q704: TD6790, PCM_4ms_Package_SOIC:SM-8, F.Cu at (354.1, 116.7)
- added R630: 47k, PCM_Resistor_SMD_AKL:R_0805_2012Metric, F.Cu at (361.2, 55.8)
- added R631: 47k, PCM_Resistor_SMD_AKL:R_0805_2012Metric, F.Cu at (361.2, 59.0)
- added R632: 47k, PCM_Resistor_SMD_AKL:R_0805_2012Metric, F.Cu at (361.2, 62.1)
- added R713: 470, PCM_Resistor_SMD_AKL:R_0805_2012Metric, F.Cu at (347.1, 80.8)
- added R714: 10k, PCM_Resistor_SMD_AKL:R_0805_2012Metric, F.Cu at (347.1, 84.0)
- added R715: 12k, PCM_Resistor_SMD_AKL:R_0805_2012Metric, F.Cu at (347.1, 87.1)
- added SW612: ENC_MENU, Alps_Rotary_Encoder:RotaryEncoder_Alps_EC11E-Switch_Vertical_H20mm_5Pin, F.Cu at (342.4, 59.4)
- added TH701: 10k, Resistor_SMD:R_0603_1608Metric, F.Cu at (351.4, 88.7)
- C706: value 100n -> 2u2
- C707, C710: value 100n -> 10u
- C708: value 10u -> 1u
- C711: value 100u -> 100n; footprint Capacitor_THT:CP_Radial_D5.0mm_P2.00mm -> Capacitor_SMD:C_0805_2012Metric; moved to F.Cu
- C712: value 10u -> 22u
- D702: value LED_CHG -> PWR
- D703: value PMEG3030 -> CHG; footprint PCM_Diode_SMD_AKL:D_SOD-123 -> LED_THT:LED_D3.0mm
- D704: value LED_PWR -> LED; footprint LED_THT:LED_D3.0mm -> LED_SMD:LED_0805_2012Metric
- L702: value 2.2uH -> 1u5; footprint Inductor_SMD:L_Changjiang_FNR4010S -> Inductor_SMD:L_Coilcraft_XAL4020-XXX
- Q701: value Q_PMOS_GSD -> BSH205G2A
- Q702: value Q_PMOS_GSD -> TD6790; footprint PCM_4ms_Package_SOT:SOT-23 -> PCM_4ms_Package_SOIC:SM-8
- R704: value 4k7 -> 3k3
- R705: value 100k -> 470
- R708: value 2M2 -> 680
- R709: value 220k -> 12k
- R710: value 680 -> 12k
- SW608: value MENU_B -> ALT_B
- TP701: value +12 -> +12A
- TP702: value -12 -> -12A
- U703: value MAX1898 -> MCP73834T
- U704: value TPS61200DRC -> TPS63021; footprint Package_SON:VSON-10-1EP_3x3mm_P0.5mm_EP1.2x2mm -> Package_SON:Texas_S-PVSON-N14
- moved D202 134.5 mm to (346.9, 136.6), turned to 0 degrees
- moved D704 133.4 mm to (353.7, 131.0), turned to 0 degrees
- moved U703 131.4 mm to (365.6, 130.1), turned to 0 degrees
- moved R710 125.4 mm to (346.2, 125.5), turned to 0 degrees
- moved C708 125.0 mm to (350.7, 128.0)
- moved J701 121.9 mm to (364.1, 122.8)
- moved C706 121.5 mm to (350.7, 122.0), turned to 0 degrees
- moved C707 119.4 mm to (350.7, 125.0), turned to 0 degrees
- moved D702 118.1 mm to (361.3, 108.0), turned to 0 degrees
- moved Q701 117.2 mm to (346.1, 129.3)
- moved J702 115.9 mm to (368.8, 122.8)
- moved TP703 113.8 mm to (350.0, 131.0), turned to 0 degrees
- moved C709 113.0 mm to (355.1, 122.0), turned to 0 degrees
- moved D703 112.3 mm to (361.3, 113.5)
- moved Q702 111.1 mm to (354.1, 109.0), turned to 0 degrees
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Connections:
- C703 pad 1: +12V -> +12VA
- C706 pad 1: Net-(U703-CT) -> VDD
- C707 pad 1: VDD -> VBATT
- C707 pad 2: Net-(Q701-G) -> GND
- C708 pad 1: BATT+ -> VCC
- C709 pad 1: SW_P -> V_PWR
- C709 pad 2: GNDPWR -> GND
- C710 pad 1: Net-(U704-VAUX) -> V_PWR
- C710 pad 2: GNDPWR -> GND
- C711 pad 1: +3.3V -> V_PWR
- C711 pad 2: GNDPWR -> GND
- C712 pad 1: +3.3V -> +3.3VP
- C712 pad 2: GNDPWR -> GND
- C713 pad 1: -12V -> -12VA
- D701 pad 1: +12V -> +12VA
- D702 pad 2: VDD -> Net-(D702-A)
- D703 pad 1: BATT+ -> Net-(D703-K)
- D704 pad 1: GND -> Net-(D704-K)
- J701 pad 1: BATT+ -> VBATT
- J702 pad 2: SW_P -> V_PWR
- L702 pad 1: SW_P -> Net-(L702-Pad1)
- L702 pad 2: Net-(U704-L) -> Net-(L702-Pad2)
- Q701 pad 1: Net-(Q701-G) -> VDD
- Q701 pad 2: Net-(D703-A) -> VBATT
- Q701 pad 3: Net-(Q701-D) -> Net-(D706-A)
- Q702 pad 1: VDD -> -12V
- Q702 pad 2: BATT+ -> unconnected-(Q702A-C1-Pad2)
- Q702 pad 3: VCC -> Net-(Q702A-B1)
- R616 pad 2: MENU_B -> ALT_B
- R702 pad 1: +12V -> +12VA
- R704 pad 1: Net-(U703-ISET) -> Net-(U703-PROG)
- R705 pad 1: VDD -> +3.3V
- R705 pad 2: GND -> Net-(D703-A)
- R706 pad 1: BATT+ -> VBATT
- R708 pad 1: Net-(U704-UVLO) -> +3.3VP
- R708 pad 2: VCC -> Net-(D704-A)
- R709 pad 1: Net-(U704-UVLO) -> +3.3VP
- R709 pad 2: GND -> Net-(Q704A-B1)
- R710 pad 1: +3.3V -> +12VA
- R710 pad 2: Net-(D704-A) -> Net-(Q703A-B1)
- SW608 pad 2: MENU_B -> ALT_B
- TP701 pad 1: +12V -> +12VA
- TP702 pad 1: -12V -> -12VA
- TP703 pad 1: BATT+ -> VBATT
- U602 pad 21: MENU_B -> ALT_B
- U603 pad 1: unconnected-(U603-GPB0-Pad1) -> MENU_B
- U603 pad 2: unconnected-(U603-GPB1-Pad2) -> ENCMENU_R
- U603 pad 3: unconnected-(U603-GPB2-Pad3) -> ENCMENU_L
- U702 pad 5: -12V -> -12VA
- U703 pad 10: Net-(Q701-D) -> VBATT
- U703 pad 2: Net-(D702-K) -> VDD
- U703 pad 3: unconnected-(U703-EN/OK-Pad3) -> Net-(D703-K)
- U703 pad 4: Net-(U703-ISET) -> Net-(D702-K)
- U703 pad 5: Net-(U703-CT) -> GND
- U703 pad 6: GND -> Net-(U703-PROG)
- U703 pad 7: BATT+ -> +3.3V
- U703 pad 8: GND -> Net-(U703-THERM)
- U703 pad 9: Net-(Q701-G) -> VBATT
- U704 pad 1: Net-(U704-VAUX) -> V_PWR
- U704 pad 10: Net-(U704-FB) -> V_PWR
- U704 pad 11: GNDPWR -> VIN
- U704 pad 2: +3.3V -> GND
- U704 pad 3: Net-(U704-L) -> (no net)
- U704 pad 4: GNDPWR -> +3.3VP
- U704 pad 5: SW_P -> unconnected-(U704-VOUT-Pad5)
- U704 pad 6: SW_P -> Net-(L702-Pad2)
- U704 pad 7: Net-(U704-UVLO) -> unconnected-(U704-L2-Pad7)
- U704 pad 8: +3.3V -> Net-(L702-Pad1)
- U704 pad 9: GND -> unconnected-(U704-L1-Pad9)
- U705 pad 5: -12V -> -12VA
Routing:
- net VDD: track 36.3 -> 0.00 mm
- net BATT+: track 34.5 -> 0.00 mm, vias 1 -> 0
- net VCC: track 33.6 -> 0.00 mm, vias 2 -> 0
- net GND: track 47.0 -> 25.8 mm, vias 20 -> 10
- net SW_P: track 15.2 -> 0.00 mm
- net +3.3V: track 28.5 -> 16.4 mm, vias 6 -> 1
- net Net-(D703-A): track 12.0 -> 0.00 mm
- net Net-(Q701-G): track 9.01 -> 0.00 mm
- net Net-(U704-FB): track 8.56 -> 0.00 mm
- net Net-(D702-K): track 7.70 -> 0.00 mm
- net Net-(Q701-D): track 6.64 -> 0.00 mm
- net Net-(D704-A): track 4.72 -> 0.00 mm
- net Net-(U703-ISET): track 4.54 -> 0.00 mm
- net Net-(U704-UVLO): track 4.32 -> 0.00 mm
- net VBUS: track 10.8 -> 6.80 mm, vias 2 -> 1
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- removed copper zone on F.Cu, net GNDPWR

Commit message: cleaned up CV opamps
Parts:
- removed C302, C303, C307, C308, C311, C312, C343, C344, C345, C346, C347, C348, C363, C364, C365, C366, C367, C368, C379, C380, C381, C382: 100n, Capacitor_SMD:C_0805_2012Metric
- removed C351, C352, C353, C354, C355, C356, C357, C360, C361, C362, C369, C370, C373, C374, C375, C376, C377, C378: 470n, Capacitor_SMD:C_0805_2012Metric
- removed D608: SK6812, LED_SMD:LED_SK6812_PLCC4_5.0x5.0mm_P3.2mm
- removed R302, R306, R308, R310, R312, R314, R317, R318, R321, R322, R324, R326: 27k, PCM_Resistor_SMD_AKL:R_0805_2012Metric
- removed R303, R305, R307, R309, R311, R313, R315, R316, R319, R320, R323, R325, R327, R328, R329, R330, R331, R332, R339, R340, R341, R342, R343, R344: 100k, PCM_Resistor_SMD_AKL:R_0805_2012Metric
- removed R333, R334, R335, R336, R337, R338, R345, R346, R347, R348, R349, R350: 56k, PCM_Resistor_SMD_AKL:R_0805_2012Metric
- removed U302, U305, U307, U310, U311, U312, U314, U315, U316, U319: TL074, Package_SO:SOIC-14_3.9x8.7mm_P1.27mm
- removed U303: TL072, Package_SO:SOIC-8_3.9x4.9mm_P1.27mm
- C625, C626, R630, R631, R632: moved to B.Cu
- R801, R802, R803, R804, R805, R806: value 47k -> 100k
- R807: value 100k -> 47k
- moved C625 179.7 mm to (181.6, 59.7), turned to 90 degrees
- moved R630 176.1 mm to (185.2, 59.7), turned to -90 degrees
- moved R632 171.4 mm to (190.2, 51.6), turned to 90 degrees
- moved R631 171.1 mm to (190.2, 59.7), turned to -90 degrees
- moved C626 169.1 mm to (192.3, 59.7), turned to 90 degrees
- moved SW612 157.3 mm to (185.2, 62.9), turned to 90 degrees
- moved C208 44.3 mm to (157.8, 89.9)
- moved C209 44.3 mm to (170.2, 89.9)
- moved U202 44.3 mm to (153.3, 95.6)
- moved U203 44.3 mm to (165.9, 95.6)
- moved U402 28.2 mm to (90.8, 131.1), turned to 0 degrees
- moved U403 28.2 mm to (117.1, 131.1), turned to 0 degrees
- moved U404 28.2 mm to (143.4, 131.1), turned to 0 degrees
- moved U405 28.2 mm to (169.7, 131.1), turned to 0 degrees
- moved U406 28.2 mm to (196.0, 131.1), turned to 0 degrees
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Connections:
- net AUDIO_OUT_L renamed AUDIO_OUT_R
- D607 pad 4: Net-(D607-DOUT) -> VOICE_PX
- U201 pad 11: unconnected-(U201-PC3-Pad11) -> FAN
- U704 pad 3: (no net) -> +3.3VP
- U801 pad 11: +12V -> -12V
- U801 pad 4: -12V -> +12V
Routing:
- net -12V: track 235.4 -> 0.00 mm
- net +12V: track 279.8 -> 78.2 mm
- net -12VA: track 0.00 -> 18.9 mm
- net Net-(L702-Pad1): track 0.00 -> 4.92 mm

Commit message: footprints placed
Parts:
- removed C383, C384: 100n, Capacitor_SMD:C_0805_2012Metric
- removed U320: TL072, Package_SO:SOIC-8_3.9x4.9mm_P1.27mm
- added C302: 100n, Capacitor_SMD:C_0805_2012Metric, F.Cu at (81.0, 122.4)
- added C303: 100n, Capacitor_SMD:C_0805_2012Metric, F.Cu at (69.4, 122.4)
- added C307: 100n, Capacitor_SMD:C_0805_2012Metric, F.Cu at (101.3, 127.1)
- added C308: 100n, Capacitor_SMD:C_0805_2012Metric, F.Cu at (112.9, 127.1)
- added C311: 100n, Capacitor_SMD:C_0805_2012Metric, F.Cu at (101.3, 115.4)
- added C312: 100n, Capacitor_SMD:C_0805_2012Metric, F.Cu at (112.8, 115.4)
- added C320: 100n, Capacitor_SMD:C_0805_2012Metric, B.Cu at (60.8, 43.5)
- added C341: 100n, Capacitor_SMD:C_0805_2012Metric, B.Cu at (49.5, 43.5)
- added C343: 100n, Capacitor_SMD:C_0805_2012Metric, F.Cu at (128.7, 115.4)
- added C344: 100n, Capacitor_SMD:C_0805_2012Metric, F.Cu at (140.3, 115.4)
- added C345: 100n, Capacitor_SMD:C_0805_2012Metric, F.Cu at (128.7, 126.4)
- added C346: 100n, Capacitor_SMD:C_0805_2012Metric, F.Cu at (140.3, 126.4)
- added C347: 100n, Capacitor_SMD:C_0805_2012Metric, F.Cu at (158.6, 116.2)
- added C348: 100n, Capacitor_SMD:C_0805_2012Metric, F.Cu at (170.0, 116.2)
- added C351: 470n, Capacitor_SMD:C_0805_2012Metric, B.Cu at (112.0, 88.1)
- added C352: 470n, Capacitor_SMD:C_0805_2012Metric, B.Cu at (110.0, 91.7)
- added C353: 470n, Capacitor_SMD:C_0805_2012Metric, B.Cu at (109.4, 76.3)
- added C354: 470n, Capacitor_SMD:C_0805_2012Metric, B.Cu at (113.7, 91.7)
- added C355: 470n, Capacitor_SMD:C_0805_2012Metric, B.Cu at (108.4, 88.1)
- added C356: 470n, Capacitor_SMD:C_0805_2012Metric, B.Cu at (112.8, 76.3)
- added C357: 470n, Capacitor_SMD:C_0805_2012Metric, B.Cu at (82.1, 88.1)
- added C360: 470n, Capacitor_SMD:C_0805_2012Metric, B.Cu at (80.2, 91.7)
- added C361: 470n, Capacitor_SMD:C_0805_2012Metric, B.Cu at (78.5, 88.1)
- added C362: 470n, Capacitor_SMD:C_0805_2012Metric, B.Cu at (83.8, 91.7)
- added C363: 100n, Capacitor_SMD:C_0805_2012Metric, F.Cu at (158.6, 127.0)
- added C364: 100n, Capacitor_SMD:C_0805_2012Metric, F.Cu at (169.9, 127.0)
- added C365: 100n, Capacitor_SMD:C_0805_2012Metric, F.Cu at (187.9, 116.2)
- added C366: 100n, Capacitor_SMD:C_0805_2012Metric, F.Cu at (199.2, 116.1)
- added C367: 100n, Capacitor_SMD:C_0805_2012Metric, F.Cu at (187.9, 128.5)
- added C368: 100n, Capacitor_SMD:C_0805_2012Metric, F.Cu at (199.3, 128.5)
- added C369: 470n, Capacitor_SMD:C_0805_2012Metric, B.Cu at (78.6, 76.3)
- added C370: 470n, Capacitor_SMD:C_0805_2012Metric, B.Cu at (82.0, 76.3)
- added C373: 470n, Capacitor_SMD:C_0805_2012Metric, B.Cu at (96.6, 76.4)
- added C374: 470n, Capacitor_SMD:C_0805_2012Metric, B.Cu at (97.1, 88.2)
- added C375: 470n, Capacitor_SMD:C_0805_2012Metric, B.Cu at (93.1, 76.3)
- added C376: 470n, Capacitor_SMD:C_0805_2012Metric, B.Cu at (93.6, 88.2)
- added C377: 470n, Capacitor_SMD:C_0805_2012Metric, B.Cu at (95.4, 91.9)
- added C378: 470n, Capacitor_SMD:C_0805_2012Metric, B.Cu at (99.1, 91.9)
- added C379: 100n, Capacitor_SMD:C_0805_2012Metric, F.Cu at (217.5, 115.3)
- added C380: 100n, Capacitor_SMD:C_0805_2012Metric, F.Cu at (228.7, 115.3)
- added C381: 100n, Capacitor_SMD:C_0805_2012Metric, F.Cu at (226.0, 124.4)
- added C382: 100n, Capacitor_SMD:C_0805_2012Metric, F.Cu at (220.5, 133.8)
- added R351: 100k, PCM_Resistor_SMD_AKL:R_0805_2012Metric, B.Cu at (60.7, 40.5)
- added R352: 27k, PCM_Resistor_SMD_AKL:R_0805_2012Metric, B.Cu at (59.2, 37.6)
- added R353: 100k, PCM_Resistor_SMD_AKL:R_0805_2012Metric, B.Cu at (60.5, 47.7)
- added R354: 27k, PCM_Resistor_SMD_AKL:R_0805_2012Metric, B.Cu at (57.5, 49.2)
- added TP704: -12V, TestPoint:TestPoint_Pad_D1.0mm_Value, F.Cu at (31.5, 156.2)
- added TP705: +12V, TestPoint:TestPoint_Pad_D1.0mm_Value, F.Cu at (37.4, 127.1)
- added TP706: 3V3P, TestPoint:TestPoint_Pad_D1.0mm_Value, F.Cu at (314.6, 49.6)
- added TP707: 3V3, TestPoint:TestPoint_Pad_D1.0mm_Value, F.Cu at (306.5, 49.7)
- added U302: TL074, Package_SO:SOIC-14_3.9x8.7mm_P1.27mm, F.Cu at (75.3, 122.4)
- added U303: TL072, Package_SO:SOIC-8_3.9x4.9mm_P1.27mm, F.Cu at (223.0, 129.1)
- added U305: TL074, Package_SO:SOIC-14_3.9x8.7mm_P1.27mm, F.Cu at (107.1, 127.1)
- added U307: TL074, Package_SO:SOIC-14_3.9x8.7mm_P1.27mm, F.Cu at (107.0, 115.4)
- added U310: TL074, Package_SO:SOIC-14_3.9x8.7mm_P1.27mm, F.Cu at (134.5, 115.4)
- added U311: TL074, Package_SO:SOIC-14_3.9x8.7mm_P1.27mm, F.Cu at (134.4, 126.4)
- added U312: TL074, Package_SO:SOIC-14_3.9x8.7mm_P1.27mm, F.Cu at (164.3, 116.2)
- added U314: TL074, Package_SO:SOIC-14_3.9x8.7mm_P1.27mm, F.Cu at (164.3, 127.0)
- added U315: TL074, Package_SO:SOIC-14_3.9x8.7mm_P1.27mm, F.Cu at (193.6, 116.2)
- added U316: TL074, Package_SO:SOIC-14_3.9x8.7mm_P1.27mm, F.Cu at (193.6, 128.5)
- added U319: TL074, Package_SO:SOIC-14_3.9x8.7mm_P1.27mm, F.Cu at (223.1, 115.3)
- added U321: TL074, Package_SO:SOIC-14_3.9x8.7mm_P1.27mm, B.Cu at (55.2, 43.4)
- C610, R501, R502, R503, R504, R505, R506, R507, R508, R509, R510, R511, R512, R513, R514, U601, U602: moved to B.Cu
- C702, C703: footprint Capacitor_THT:CP_Radial_D4.0mm_P2.00mm -> Capacitor_SMD:C_0805_2012Metric; moved to F.Cu
- D704: value LED -> SMPS
- moved C715 323.9 mm to (25.4, 138.3), turned to -90 degrees
- moved Q703 323.7 mm to (32.0, 133.1), turned to 180 degrees
- moved R710 320.9 mm to (25.4, 134.1), turned to -90 degrees
- moved Q702 316.9 mm to (39.1, 144.5), turned to 90 degrees
- moved C718 315.4 mm to (34.1, 148.0), turned to 180 degrees
- moved JP703 312.6 mm to (32.7, 127.1), turned to 180 degrees
- moved R715 312.1 mm to (39.2, 138.1)
- moved C716 309.5 mm to (38.4, 133.1), turned to -90 degrees
- moved C717 305.4 mm to (42.9, 138.1)
- moved JP704 303.4 mm to (43.8, 142.0), turned to -90 degrees
- moved D202 135.3 mm to (294.7, 11.8), turned to 90 degrees
- moved TP703 131.5 mm to (312.7, 4.95)
- moved U703 130.7 mm to (305.2, 14.2)
- moved J701 126.9 mm to (317.1, 4.91)
- moved D703 122.0 mm to (306.5, 4.51)
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Connections:
- net DISP_LST renamed DISP_RST
- net MIDI_LX renamed MIDI_RX
- C301 pad 1: +3.3VA -> +3.3V
- C304 pad 1: +3.3VA -> +3.3V
- R304 pad 1: +3.3VA -> +3.3V
- U301 pad 13: LVL2_DAC -> Net-(U301-VOUTB)
- U301 pad 3: +3.3VA -> +3.3V
- U301 pad 4: LVL1_DAC -> Net-(U301-VOUTA)
- U501 pad 1: MD_8 -> MD_1
- U501 pad 2: MD_7 -> MD_2
- U501 pad 3: MD_6 -> MD_3
- U501 pad 4: MD_5 -> MD_4
- U501 pad 5: MD_4 -> MD_5
- U501 pad 6: MD_3 -> MD_6
- U501 pad 7: MD_2 -> MD_7
- U501 pad 8: MD_1 -> MD_8
- U602 pad 1: ENCA_L -> ENCD_R
- U602 pad 2: ENCA_R -> ENCD_L
- U602 pad 21: ALT_B -> ENV1_B
- U602 pad 22: MIX2_B -> ENV2_B
- U602 pad 23: MIX1_B -> LFO1_B
- U602 pad 24: LFO3_B -> LFO2_B
- U602 pad 25: LFO2_B -> LFO3_B
- U602 pad 26: LFO1_B -> MIX1_B
- U602 pad 27: ENV2_B -> MIX2_B
- U602 pad 28: ENV1_B -> ALT_B
- U602 pad 3: ENCB_L -> ENCC_R
- U602 pad 4: ENCB_R -> ENCC_L
- U602 pad 5: ENCC_L -> ENCB_R
- U602 pad 6: ENCC_R -> ENCB_L
- U602 pad 7: ENCD_L -> ENCA_R
- U602 pad 8: ENCD_R -> ENCA_L
- U704 pad 11: VIN -> V_PWR
- U704 pad 5: unconnected-(U704-VOUT-Pad5) -> +3.3VP
- U704 pad 7: unconnected-(U704-L2-Pad7) -> Net-(L702-Pad2)
- U704 pad 9: unconnected-(U704-L1-Pad9) -> Net-(L702-Pad1)
Routing:
- net +12V: track 78.2 -> 0.00 mm
- net USB_D+: track 57.5 -> 83.3 mm
- net USB_D-: track 60.7 -> 86.1 mm
- net -12VA: track 18.9 -> 0.00 mm
- net +3.3V: track 16.4 -> 0.00 mm, vias 1 -> 0
- net GND: track 25.8 -> 14.1 mm, vias 10 -> 3
- net Net-(D701-A): track 8.20 -> 0.00 mm
- net Net-(U701-FB): track 6.14 -> 0.00 mm
- net Net-(L702-Pad1): track 4.92 -> 0.00 mm
- net Net-(JP701-A): track 4.29 -> 0.00 mm
- net Net-(JP702-A): track 4.09 -> 0.00 mm
- net Net-(U701-Vc): track 3.51 -> 0.00 mm
- net Net-(U705-CAP+): track 2.71 -> 0.00 mm
- net Net-(U702-CAP+): track 2.69 -> 0.00 mm
- net Net-(U705-CAP-): track 2.61 -> 0.00 mm
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Other:
- board text added: "BOOT"
- board text added: "RST"
