File: PolySynthMotherboard/PolySynthMotherboard.kicad_sch (KiCad schematic)
At the start: 0 parts

Commit message: motherboard hardware
Other:
- added sheet CV Outputs (CVOutputs.kicad_sch)
- added sheet VoiceBoards (Voices.kicad_sch)
Changed lines of the file:
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@@
+    )
+  )
+  (sheet (at 59.944 17.272) (size 36.068 29.972) (fields_autoplaced)
+    (stroke (width 0.1524) (type solid))
+    (fill (color 0 0 0 0.0000))
+    (property "Sheetname" "CV Outputs" (at 59.944 16.5604 0)
+      (effects (font (size 1.27 1.27)) (justify left bottom))
+    )
+    (property "Sheetfile" "CVOutputs.kicad_sch" (at 59.944 47.8286 0)
+      (effects (font (size 1.27 1.27)) (justify left top))
+    )
+    (instances
+      (project "PolySynthMotherboard"
+        (path "/22649217-9810-470f-bc7b-6f743ad2b90e" (page "3"))
+      )
+    )
+  )
+  (sheet (at 17.272 52.578) (size 40.64 27.686) (fields_autoplaced)
+    (stroke (width 0.1524) (type solid))
+    (fill (color 0 0 0 0.0000))
+    (property "Sheetname" "VoiceBoards" (at 17.272 51.8664 0)
+      (effects (font (size 1.27 1.27)) (justify left bottom))
+    )
+    (property "Sheetfile" "Voices.kicad_sch" (at 17.272 80.8486 0)
+      (effects (font (size 1.27 1.27)) (justify left top))
+    )
+    (instances
+      (project "PolySynthMotherboard"
+        (path "/22649217-9810-470f-bc7b-6f743ad2b90e" (page "4"))
+      )
     )
   )

Commit message: power supply/ output circuits
Other:
- added sheet AudioOut (AudioOut.kicad_sch)
- added sheet Controls (Controls.kicad_sch)
- added sheet ModMatrix (ModMatrix.kicad_sch)
- added sheet PowerSupply (PowerSupply.kicad_sch)
Changed lines of the file:
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@@
 (kicad_sch (version 20230121) (generator eeschema)
   (paper "A4")
+  (sheet (at 97.7392 53.1368) (size 38.2016 27.7368) (fields_autoplaced)
+    (stroke (width 0.1524) (type solid))
+    (fill (color 0 0 0 0.0000))
+    (property "Sheetname" "PowerSupply" (at 97.7392 52.4252 0)
+      (effects (font (size 1.27 1.27)) (justify left bottom))
+    )
+    (property "Sheetfile" "PowerSupply.kicad_sch" (at 97.7392 81.4582 0)
+      (effects (font (size 1.27 1.27)) (justify left top))
+    )
+    (instances
+      (project "PolySynthMotherboard"
+        (path "/22649217-9810-470f-bc7b-6f743ad2b90e" (page "7"))
+      )
+    )
+  )
   (sheet (at 17.272 17.272) (size 40.386 29.845) (fields_autoplaced)
     (stroke (width 0.1524) (type solid))
@@
       (project "PolySynthMotherboard"
         (path "/22649217-9810-470f-bc7b-6f743ad2b90e" (page "2"))
+      )
+    )
+  )
+  (sheet (at 59.944 53.086) (size 36.068 27.432) (fields_autoplaced)
+    (stroke (width 0.1524) (type solid))
+    (fill (color 0 0 0 0.0000))
+    (property "Sheetname" "ModMatrix" (at 59.944 52.3744 0)
+      (effects (font (size 1.27 1.27)) (justify left bottom))
+    )
+    (property "Sheetfile" "ModMatrix.kicad_sch" (at 59.944 81.1026 0)
+      (effects (font (size 1.27 1.27)) (justify left top))
+    )
+    (instances
+      (project "PolySynthMotherboard"
+        (path "/22649217-9810-470f-bc7b-6f743ad2b90e" (page "5"))
+      )
+    )
+  )
+  (sheet (at 17.399 85.09) (size 40.894 27.432) (fields_autoplaced)
+    (stroke (width 0.1524) (type solid))
+    (fill (color 0 0 0 0.0000))
+    (property "Sheetname" "AudioOut" (at 17.399 84.3784 0)
+      (effects (font (size 1.27 1.27)) (justify left bottom))
+    )
+    (property "Sheetfile" "AudioOut.kicad_sch" (at 17.399 113.1066 0)
+      (effects (font (size 1.27 1.27)) (justify left top))
+    )
+    (instances
+      (project "PolySynthMotherboard"
+        (path "/22649217-9810-470f-bc7b-6f743ad2b90e" (page "8"))
       )
     )
@@
       )
     )
+  )
+  (sheet (at 97.536 17.272) (size 38.354 29.972) (fields_autoplaced)
+    (stroke (width 0.1524) (type solid))
+    (fill (color 0 0 0 0.0000))
+    (property "Sheetname" "Controls" (at 97.536 16.5604 0)
+      (effects (font (size 1.27 1.27)) (justify left bottom))
+    )
+    (property "Sheetfile" "Controls.kicad_sch" (at 97.536 47.8286 0)
+      (effects (font (size 1.27 1.27)) (justify left top))
+    )
+    (instances
+      (project "PolySynthMotherboard"
+        (path "/22649217-9810-470f-bc7b-6f743ad2b90e" (page "6"))
+      )
+    )

Commit message: added terminations
Other:
- removed sheet PowerSupply
Changed lines of the file:
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@@
 	(paper "A4")
-	(sheet
-		(at 97.7392 53.1368)
-		(size 38.2016 27.7368)
-		(fields_autoplaced yes)
-		(stroke
-			(width 0.1524)
-			(type solid)
-		)
-		(fill
-			(color 0 0 0 0.0000)
-		)
-		(property "Sheetname" "PowerSupply"
-			(at 97.7392 52.4252 0)
-			(effects
-				(font
-					(size 1.27 1.27)
-				)
-				(justify left bottom)
-			)
-		)
-		(property "Sheetfile" "PowerSupply.kicad_sch"
-			(at 97.7392 81.4582 0)
-			(effects
-				(font
-					(size 1.27 1.27)
-				)
-				(justify left top)
-			)
-		)
-		(instances
-			(project "PolySynthMotherboard"
-				(path "/22649217-9810-470f-bc7b-6f743ad2b90e"
-					(page "7")
-				)
-			)
-		)
-	)
 	(sheet
 		(at 17.272 17.272)
@@
 	)
 	(sheet
-		(at 17.399 85.09)
-		(size 40.894 27.432)
+		(at 97.663 53.086)
+		(size 37.973 27.432)
 		(fields_autoplaced yes)
 		(stroke
@@
 		)
 		(property "Sheetname" "AudioOut"
-			(at 17.399 84.3784 0)
+			(at 97.663 52.3744 0)
 			(effects
 				(font
@@
 		)
 		(property "Sheetfile" "AudioOut.kicad_sch"
-			(at 17.399 113.1066 0)
+			(at 97.663 81.1026 0)
 			(effects
 				(font
