File: PolySynthSplitBoard/PolySynthSplitBoard.kicad_pcb (KiCad board)
At the start: 4 copper layers, 441 parts, among them J201 AUDIO_OUT, J401 PWR, J402 DATA, J403 SWD Header, J404 MIDI_In, J405 Micro_SD_Card_Det2, J406 MIDI_Out, J407 MIDI_Thru, J801 A_UPPER, J802 B_UPPER, J803 C_UPPER, J901 A_LOWER, J902 B_LOWER, J903 C_LOWER, SW401 RST, SW402 BOOT, SW501 SB, SW502 MS1, SW503 MD1, SW504 MS2, SW505 MD2, SW506 MS3, SW507 MD3, SW508 MS4, SW509 MD4, SW510 MS5, SW511 MD5, SW512 MS6, SW513 MD6, SW514 MD7, SW515 MD8, SW601 ENV1_B, SW602 ENV2_B, SW603 HP_B, SW604 LFO1_B, SW605 LFO2_B, SW606 HP_B, SW607 LFO3_B, SW608 FF_B, SW609 MIX1_B, SW610 MIX2_B, SW611 ENC_MENU, SW612 ALT_B, U201 TL074, U301 DAC7578xPW, U302 TL074, U303 TL072, U304 TL074, U305 TL072, U306 TMUX4051, U307 TL074, U308 TMUX4051, U309 TL072, U310 TL074, U311 TL072, U312 TL074, U313 TMUX4051, U314 TMUX4051, U315 TL074, U316 TL074, U317 TL074, U318 TL072, U319 TL072, U320 TL072, U321 TMUX4051, U322 TMUX4051, U323 TMUX4051, U401 STM32F411RETx, U402 74HC595, U403 74HC595, U404 74HC04, U405 6N138, U501 MCP23S17_SS, U601 MCP23S17_SS, U602 MCP23S17_SS, U603 ILI9341, U701 TCA9548APWR, U702 V1, U703 V4, U704 V2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

Commit message: upper board routing
Parts:
- C604, C605, C606, C607, C608, C609, C610, C611, C612, C613, C614, C615, C618, C619, C620, C621, C622, C623, C624, C625, C626, R601, R602, R603, R604, R605, R606, R607, R608, R609, R610, R611, R612, R613, R614, R615, R616, R617, R618, R619, R620, R621, R622, R625, R626, R627, R628, R629, R630, R631, R632, R633, R634, R635, R636, R637, R638, R639, U601, U602: moved to B.Cu
- RE603: value ENC_LES -> ENC_RES
- moved J902 479.0 mm to (5.00, 119.0)
- moved SW612 270.4 mm to (10.7, 77.6)
- moved J803 259.0 mm to (305.0, 60.0)
- moved R639 249.9 mm to (14.7, 81.2), turned to -90 degrees
- moved R636 249.7 mm to (11.4, 65.8), turned to -90 degrees
- moved R633 245.7 mm to (16.4, 58.0), turned to 90 degrees
- moved R638 242.6 mm to (16.4, 65.8), turned to -90 degrees
- moved C624 235.1 mm to (11.4, 72.4), turned to -90 degrees
- moved R637 233.1 mm to (20.4, 48.6)
- moved R634 230.4 mm to (20.6, 33.3)
- moved C625 229.3 mm to (16.4, 72.4), turned to -90 degrees
- moved J801 225.3 mm to (305.0, 8.00)
- moved R604 223.9 mm to (26.4, 71.3), turned to -90 degrees
- moved SW601 218.6 mm to (19.3, 10.9)
- moved R607 215.1 mm to (31.4, 71.3), turned to -90 degrees
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Connections:
- R631 pad 2: EXP_INTR_A_U -> EXP_INTR_B_U
- R632 pad 2: EXP_INTR_B_U -> EXP_INTR_A_U
- U602 pad 4: PWMTOG_B -> ENCDEPTH_L
- U602 pad 5: HPMODE_B -> ENCDEPTH_R
- U602 pad 6: FF_B -> PWMTOG_B
- U602 pad 7: ENCDEPTH_R -> HPMODE_B
- U602 pad 8: ENCDEPTH_L -> FF_B
Routing:
- net EXP_MOSI_U: track 0.00 -> 508.5 mm
- net EXP_SCK_U: track 0.00 -> 504.7 mm
- net EXP_MISO_U: track 0.00 -> 502.9 mm
- net EXP_CS_U: track 0.00 -> 500.4 mm
- net EXP_INTR_C_U: track 0.00 -> 296.3 mm, vias 0 -> 1
- net ENCMENU_L: track 0.00 -> 291.5 mm
- net ENCMENU_R: track 0.00 -> 286.6 mm
- net MENU_B: track 0.00 -> 282.3 mm
- net VOICE_PX: track 0.00 -> 232.9 mm
- net PIXELS_MATRIX_U: track 0.00 -> 219.2 mm
- net PIXELS_MAIN_U: track 0.00 -> 216.6 mm, vias 0 -> 1
- net GNDA: track 0.00 -> 184.0 mm, vias 0 -> 101
- net FF_B: track 0.00 -> 121.1 mm, vias 0 -> 1
- net EXP_INTR_B_U: track 0.00 -> 120.4 mm
- net EXP_INTR_A_U: track 0.00 -> 118.3 mm
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- added copper zone on F.Cu, net +3.3VP
- added copper zone on In1.Cu, net GNDA
- added copper zone on In2.Cu, net GNDA
Other:
- board text removed: "Lower>"
- board text removed: "Upper>"
