File: PolySynthSplitBoard/CVOutputs.kicad_sch (KiCad schematic)
At the start: 132 parts, among them U301 DAC7578xPW, U302 TL074, U303 TL072, U304 TL074, U305 TL072, U306 TMUX4051, U307 TL074, U308 TMUX4051, U309 TL072, U310 TL074, U311 TL072, U312 TL074, U313 TMUX4051, U314 TMUX4051, U315 TL074, U316 TL074, U317 TL074, U318 TL072, U319 TL072, U320 TL072, U321 TMUX4051, U322 TMUX4051, U323 TMUX4051

Commit message: motherboard rev2 passing DRC
Parts:
- TP301: value TestPoint -> LVL1_DAC
- TP302: value TestPoint -> LVL2_DAC
- TP303: value TestPoint -> PWM2_DAC
- TP304: value TestPoint -> VCA_DAC
- TP305: value TestPoint -> PWM1_DAC
- TP306: value TestPoint -> FOLD_DAC
- TP307: value TestPoint -> CTF_DAC
- TP308: value TestPoint -> CTF_RAW
- TP309: value TestPoint -> LVL1_RAW
- TP310: value TestPoint -> LVL2_RAW
Changed lines of the file:
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@@
 			)
 		)
-		(property "Value" "TestPoint"
+		(property "Value" "FOLD_DAC"
 			(at 95.25 214.3759 0)
 			(effects
@@
 			)
 		)
-		(property "Value" "TestPoint"
+		(property "Value" "LVL1_DAC"
 			(at 92.71 172.7199 0)
 			(effects
@@
 			)
 		)
-		(property "Value" "TestPoint"
+		(property "Value" "LVL2_RAW"
 			(at 69.85 213.3599 0)
 			(effects
@@
 			)
 		)
-		(property "Value" "TestPoint"
+		(property "Value" "CTF_RAW"
 			(at 71.12 196.5959 0)
 			(effects
@@
 			)
 		)
-		(property "Value" "TestPoint"
+		(property "Value" "CTF_DAC"
 			(at 95.25 224.0279 0)
 			(effects
@@
 			)
 		)
-		(property "Value" "TestPoint"
+		(property "Value" "LVL2_DAC"
 			(at 92.71 181.8639 0)
 			(effects
@@
 			)
 		)
-		(property "Value" "TestPoint"
+		(property "Value" "VCA_DAC"
 			(at 93.98 198.3739 0)
 			(effects
@@
 			)
 		)
-		(property "Value" "TestPoint"
+		(property "Value" "PWM2_DAC"
 			(at 93.98 189.4839 0)
 			(effects
@@
 			)
 		)
-		(property "Value" "TestPoint"
+		(property "Value" "LVL1_RAW"
 			(at 69.85 204.7239 0)
 			(effects
@@
 			)
 		)
-		(property "Value" "TestPoint"
+		(property "Value" "PWM1_DAC"
 			(at 95.25 206.2479 0)
 			(effects
