File: VoiceBoardR4/DCO.kicad_sch (KiCad schematic)
At the start: 83 parts, among them Q201 BC857, Q202 BC857, U201 TL074, U202 TL074, U203 MCP4451-104E-ST, U204 TL074, U205 MCP4451-104E-ST, U206 TL074

Commit message: voice rev4 passing DRC
Parts:
- added OSC1: OSC1, TestPoint:TestPoint_THTPad_D1.0mm_Drill0.5mm, symbol Connector:TestPoint
- added OSC2, OSCMIX1: OSC2, TestPoint:TestPoint_THTPad_D1.0mm_Drill0.5mm, symbol Connector:TestPoint
- R225: value 92k -> 100k
- R226: value 100k -> 47k
- R245: value 56k -> 33k
Connections:
- net GND: now also U206.10 (+); no longer U206.3 (+)
- net OSC_MIX: now also OSCMIX1.1
- net PWM_1_CV: now also U206.3 (+); no longer U206.5 (+)
- net PWM_2_CV: now also U206.5 (+); no longer U206.10 (+)
- net SAW1_FULL: now also U206.2 (-); no longer U206.6 (-)
- net SAW2_FULL: now also U206.6 (-); no longer U206.9 (-)
- net at U206.8: now also R245.2, R246.1; no longer D206.2 (A)
- net at R242.2, R244.2, R245.1: now also U206.9 (-); no longer U206.2 (-)
- net O2_MIXF: now reaches R231.2, U203.13 (P0B), U204.7
- net O2_MIXF: now also OSC2.1
- net at D205.2 (A): now also U206.1; no longer U206.7
- net O1_MIXF: now reaches R241.2, U204.8, U205.13 (P0B)
- net O1_MIXF: now also OSC1.1
- new net: D206.2 (A), U206.7
Other:
- note removed: "The decouplig caps and inverting amp here give us a 6Vpp AC signal"
- moved on the sheet: C211, U205A, U206A, U206B, U206C
