File: VoiceBoardR4/Filter.kicad_sch (KiCad schematic)
At the start: 40 parts, among them Q301 BC857, Q302 BC857, U301 TL074, U302 AD5280, U303 LM13700, U304 DI79L05ZAB, U305 DI78L05ZAB

Commit message: voice rev4 passing DRC
Parts:
- added C315: 100n, Capacitor_SMD:C_0805_2012Metric, symbol Device:C
Connections:
- net +3.3V: now also C315.1
- net GND: now also U301.5 (+), C315.2; no longer U301.3 (+)
- net at C306.2, D301.1 (K), D302.2 (A)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: now also U301.8; no longer U301.14
- net at D301.2 (A), D302.1 (K), R315.1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: now also U301.9 (-); no longer U301.13 (-)
- net at C306.1, U303.12: now also U301.3 (+); no longer U301.5 (+)
- net at C301.2, Q301.3 (C), R302.2: now also U301.6 (-); no longer U301.2 (-)
- net at C305.1, R312.2: now also U301.13 (-), U301.14; no longer U301.8, U301.9 (-)
- net at C301.1, R301.2: now also U301.7; no longer U301.1
- net at R305.2, R308.2: now also U301.1, U301.2 (-); no longer U301.6 (-), U301.7
- net at C307.1, U303.5: now also U301.12 (+); no longer U301.10 (+)
- net at U302.2 (W): now also U301.10 (+); no longer U301.12 (+)
Other:
- moved on the sheet: U301A, U301B, U301C, U301D
