File: VoiceBoardR5/VoiceBoardR5.kicad_pcb (KiCad board)
At the start: 4 copper layers, 130 x 50 mm, 179 parts, among them Q201 BC857, Q202 BC857, Q301 BC857, Q302 BC857, Q401 BC857, Q402 BC857, Q403 BC847, Q404 BC857, Q405 BC847, Q406 BC857, Q407 BC857, U101 TMUX4053, U102 TMUX4053, U103 VoiceBoardConn_20P_200P, U201 TL074, U202 TL074, U203 MCP4451-104E-ST, U204 TL074, U205 MCP4451-104E-ST, U206 TL074, U301 TL074, U302 AD5280, U303 LM13700, U402 LM13700, U403 TL074, U404 TL074

Commit message: voice rev5 sent to fab
Routing:
- net +3.3V: track 172.2 -> 168.2 mm
- net +5V: track 107.6 -> 110.5 mm
- net PULSE2_FULL: track 39.6 -> 37.6 mm
- net GND: track 114.3 -> 113.7 mm, vias 84 -> 182
- net Net-(U302-~{SHDN}): track 22.4 -> 21.9 mm
- net Net-(R409-Pad1): track 6.03 -> 5.48 mm
