File: SplitBoard8Voice/CVOutputs.kicad_sch (KiCad schematic)
At the start: 132 parts, among them U301 DAC7578xPW, U302 TL074, U303 TL072, U304 TL074, U305 TL072, U306 TMUX4051, U307 TL074, U308 TMUX4051, U309 TL072, U310 TL074, U311 TL072, U312 TL074, U313 TMUX4051, U314 TMUX4051, U315 TL074, U316 TL074, U317 TL074, U318 TL072, U319 TL072, U320 TL072, U321 TMUX4051, U322 TMUX4051, U323 TMUX4051

Commit message: 8 voice schematics start
Parts:
- removed U303, U305, U311, U318, U319, U320: TL072, Package_SO:SOIC-8_3.9x4.9mm_P1.27mm, symbol Amplifier_Operational:TL072
- added C389, C390, C391, C392, C393, C394, C395, C396, C397, C398, C399, C400: 470n, Capacitor_SMD:C_0805_2012Metric, symbol Device:C
- added U303, U305, U311, U318, U319, U320: TL074, symbol Amplifier_Operational:TL074
Connections:
- net +12V: now also U303.4 (V+), U305.4 (V+), U311.4 (V+), U318.4 (V+), U319.4 (V+), U320.4 (V+)
- net -12V: now also U303.11 (V-), U305.11 (V-), U311.11 (V-), U318.11 (V-), U319.11 (V-), U320.11 (V-)
- net A5_C: now also U319.3 (+)
- net A6_C: now also U319.5 (+)
- net C5_C: now also U318.3 (+)
- net C6_C: now also U318.5 (+)
- net CUTOFF_V5: now also U318.1, U318.2 (-)
- net CUTOFF_V6: now also U318.6 (-), U318.7
- net FOLD_V5: now also U320.1, U320.2 (-)
- net FOLD_V6: now also U320.6 (-), U320.7
- net FV5_C: now also U320.3 (+)
- net FV6_C: now also U320.5 (+)
- net GND: now also C389.2, C390.2, C391.2, C392.2, C393.2, C394.2, C395.2, C396.2, C397.2, C398.2, C399.2, C400.2
- net L1V5_C: now also U305.3 (+)
- net L1V6_C: now also U305.5 (+)
- net L2V5_C: now also U303.3 (+)
- net L2V6_C: now also U303.5 (+)
- net LVL1_V5: now also U305.1, U305.2 (-)
- net LVL1_V6: now also U305.6 (-), U305.7
- net LVL2_V5: now also U303.1, U303.2 (-)
- net LVL2_V6: now also U303.6 (-), U303.7
- net P2V5_C: now also U311.3 (+)
- net P2V6_C: now also U311.5 (+)
- net PWM2_V5: now also U311.1, U311.2 (-)
- net PWM2_V6: now also U311.6 (-), U311.7
- net VCA_V5: now also U319.1, U319.2 (-)
- net VCA_V6: now also U319.6 (-), U319.7
- net A7_C: now reaches U323.2 (X6)
- net A7_C: now also C395.1, U319.10 (+)
- net A8_C: now reaches U323.4 (X7)
- net A8_C: now also C396.1, U319.12 (+)
- net L2V7_C: now reaches U306.2 (X6)
- net L2V7_C: now also C393.1, U303.10 (+)
- net L2V8_C: now reaches U306.4 (X7)
- net L2V8_C: now also C394.1, U303.12 (+)
- net FV7_C: now reaches U321.2 (X6)
- net FV7_C: now also C397.1, U320.10 (+)
- net FV8_C: now reaches U321.4 (X7)
- net FV8_C: now also C398.1, U320.12 (+)
- net L1V7_C: now reaches U308.2 (X6)
- net L1V7_C: now also C391.1, U305.10 (+)
- net L1V8_C: now reaches U308.4 (X7)
- net L1V8_C: now also C392.1, U305.12 (+)
- net C7_C: now reaches U322.2 (X6)
- net C7_C: now also C399.1, U318.10 (+)
- net C8_C: now reaches U322.4 (X7)
- net C8_C: now also C400.1, U318.12 (+)
- net P2V7_C: now reaches U313.2 (X6)
- net P2V7_C: now also C389.1, U311.10 (+)
- net P2V8_C: now reaches U313.4 (X7)
- net P2V8_C: now also C390.1, U311.12 (+)
- new net CUTOFF_V7: U318.13 (-), U318.14, U318.8, U318.9 (-)
- new net FOLD_V7: U320.8, U320.9 (-)
- new net FOLD_V8: U320.13 (-), U320.14
- new net LVL1_V7: U305.8, U305.9 (-)
- new net LVL1_V8: U305.13 (-), U305.14
- new net LVL2_V7: U303.13 (-), U303.14, U303.8, U303.9 (-)
- new net PWM2_V7: U311.8, U311.9 (-)
- new net PWM2_V8: U311.13 (-), U311.14
- new net VCA_V7: U319.8, U319.9 (-)
- new net VCA_V8: U319.13 (-), U319.14
- no-connect marks 15 -> 1
Other:
- note added: "Folder & Filter"
- note added: "VCA"
- note removed: "Folder, Filter, VCA"
- moved on the sheet: C305, C306, C307, C308, C311, C312, C313, C314, C315, C316, C317, C318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

Commit message: galaxy brain clock logic circuit
Parts:
- U303, U305, U311, U318, U319, U320: footprint (none) -> Package_SO:SOIC-14_3.9x8.7mm_P1.27mm
Changed lines of the file:
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@@
 			)
 		)
-		(property "Footprint" ""
+		(property "Footprint" "Package_SO:SOIC-14_3.9x8.7mm_P1.27mm"
 			(at 432.562 319.786 0)
 			(effects
@@
 			)
 		)
-		(property "Footprint" ""
+		(property "Footprint" "Package_SO:SOIC-14_3.9x8.7mm_P1.27mm"
 			(at 594.868 156.464 0)
 			(effects
@@
 			)
 		)
-		(property "Footprint" ""
+		(property "Footprint" "Package_SO:SOIC-14_3.9x8.7mm_P1.27mm"
 			(at 113.538 341.63 0)
 			(effects
@@
 			)
 		)
-		(property "Footprint" ""
+		(property "Footprint" "Package_SO:SOIC-14_3.9x8.7mm_P1.27mm"
 			(at 58.166 336.296 0)
 			(effects
@@
 			)
 		)
-		(property "Footprint" ""
+		(property "Footprint" "Package_SO:SOIC-14_3.9x8.7mm_P1.27mm"
 			(at 574.294 262.382 0)
 			(effects
@@
 			)
 		)
-		(property "Footprint" ""
+		(property "Footprint" "Package_SO:SOIC-14_3.9x8.7mm_P1.27mm"
 			(at 298.196 196.342 0)
 			(effects
@@
 			)
 		)
-		(property "Footprint" ""
+		(property "Footprint" "Package_SO:SOIC-14_3.9x8.7mm_P1.27mm"
 			(at 209.804 135.382 0)
 			(effects
@@
 			)
 		)
-		(property "Footprint" ""
+		(property "Footprint" "Package_SO:SOIC-14_3.9x8.7mm_P1.27mm"
 			(at 433.07 366.268 0)
 			(effects
@@
 			)
 		)
-		(property "Footprint" ""
+		(property "Footprint" "Package_SO:SOIC-14_3.9x8.7mm_P1.27mm"
 			(at 354.584 336.55 0)
 			(effects
@@
 			)
 		)
-		(property "Footprint" ""
+		(property "Footprint" "Package_SO:SOIC-14_3.9x8.7mm_P1.27mm"
 			(at 297.942 132.588 0)
 			(effects
@@
 			)
 		)
-		(property "Footprint" ""
+		(property "Footprint" "Package_SO:SOIC-14_3.9x8.7mm_P1.27mm"
 			(at 298.45 376.174 0)
 			(effects
@@
 			)
 		)
-		(property "Footprint" ""
+		(property "Footprint" "Package_SO:SOIC-14_3.9x8.7mm_P1.27mm"
 			(at 454.66 345.948 0)
 			(effects
@@
 			)
 		)
-		(property "Footprint" ""
+		(property "Footprint" "Package_SO:SOIC-14_3.9x8.7mm_P1.27mm"
 			(at 137.414 360.426 0)
 			(effects
@@
 			)
 		)
-		(property "Footprint" ""
+		(property "Footprint" "Package_SO:SOIC-14_3.9x8.7mm_P1.27mm"
 			(at 298.196 396.494 0)
 			(effects
@@
 			)
 		)
-		(property "Footprint" ""
+		(property "Footprint" "Package_SO:SOIC-14_3.9x8.7mm_P1.27mm"
 			(at 297.942 175.768 0)
 			(effects
@@
 			)
 		)
-		(property "Footprint" ""
+		(property "Footprint" "Package_SO:SOIC-14_3.9x8.7mm_P1.27mm"
 			(at 452.628 386.334 0)
 			(effects
@@
 			)
 		)
-		(property "Footprint" ""
+		(property "Footprint" "Package_SO:SOIC-14_3.9x8.7mm_P1.27mm"
 			(at 575.31 137.922 0)
 			(effects
@@
 			)
 		)
-		(property "Footprint" ""
+		(property "Footprint" "Package_SO:SOIC-14_3.9x8.7mm_P1.27mm"
 			(at 597.154 312.42 0)
 			(effects
@@
 			)
 		)
-		(property "Footprint" ""
+		(property "Footprint" "Package_SO:SOIC-14_3.9x8.7mm_P1.27mm"
 			(at 596.646 275.59 0)
 			(effects
@@
 			)
 		)
-		(property "Footprint" ""
+		(property "Footprint" "Package_SO:SOIC-14_3.9x8.7mm_P1.27mm"
 			(at 298.45 330.454 0)
 			(effects
@@
 			)
 		)
-		(property "Footprint" ""
+		(property "Footprint" "Package_SO:SOIC-14_3.9x8.7mm_P1.27mm"
 			(at 115.316 309.372 0)
 			(effects
@@
 			)
 		)
-		(property "Footprint" ""
+		(property "Footprint" "Package_SO:SOIC-14_3.9x8.7mm_P1.27mm"
 			(at 208.28 307.086 0)
 			(effects
@@
 			)
 		)
-		(property "Footprint" ""
+		(property "Footprint" "Package_SO:SOIC-14_3.9x8.7mm_P1.27mm"
 			(at 574.04 294.386 0)
 			(effects
@@
 			)
 		)
-		(property "Footprint" ""
+		(property "Footprint" "Package_SO:SOIC-14_3.9x8.7mm_P1.27mm"
 			(at 575.818 104.14 0)
 			(effects
@@
 			)
 		)
-		(property "Footprint" ""
+		(property "Footprint" "Package_SO:SOIC-14_3.9x8.7mm_P1.27mm"
 			(at 298.45 354.584 0)
 			(effects
@@
 			)
 		)
-		(property "Footprint" ""
+		(property "Footprint" "Package_SO:SOIC-14_3.9x8.7mm_P1.27mm"
 			(at 596.9 118.364 0)
 			(effects
@@
 			)
 		)
-		(property "Footprint" ""
+		(property "Footprint" "Package_SO:SOIC-14_3.9x8.7mm_P1.27mm"
 			(at 514.858 124.46 0)
 			(effects
@@
 			)
 		)
-		(property "Footprint" ""
+		(property "Footprint" "Package_SO:SOIC-14_3.9x8.7mm_P1.27mm"
 			(at 511.048 271.526 0)
 			(effects
@@
 			)
 		)
-		(property "Footprint" ""
+		(property "Footprint" "Package_SO:SOIC-14_3.9x8.7mm_P1.27mm"
 			(at 297.942 154.178 0)
 			(effects
@@
 			)
 		)
-		(property "Footprint" ""
+		(property "Footprint" "Package_SO:SOIC-14_3.9x8.7mm_P1.27mm"
 			(at 136.398 323.596 0)
 			(effects

Commit message: Eurorack power capability sorted out
Parts:
- removed U309: TL072, Package_SO:SOIC-8_3.9x4.9mm_P1.27mm, symbol Amplifier_Operational:TL072
- added C415, C416: 470n, Capacitor_SMD:C_0805_2012Metric, symbol Device:C
- added U309: TL074, Package_SO:SOIC-14_3.9x8.7mm_P1.27mm, symbol Amplifier_Operational:TL074
Connections:
- net +12V: now also U309.4 (V+)
- net -12V: now also C360.2, U309.11 (V-); no longer C360.1
- net A6_C: now also U319.12 (+); no longer U319.5 (+)
- net A7_C: now also U319.5 (+); no longer U319.10 (+)
- net A8_C: now also U319.10 (+); no longer U319.12 (+)
- net C6_C: now also U318.12 (+); no longer U318.5 (+)
- net C7_C: now also U318.5 (+); no longer U318.10 (+)
- net C8_C: now also U318.10 (+); no longer U318.12 (+)
- net CUTOFF_V6: now also U318.13 (-), U318.14; no longer U318.6 (-), U318.7
- net CUTOFF_V7: now also U318.6 (-), U318.7; no longer U318.13 (-), U318.14
- net FOLD_V6: now also U320.13 (-), U320.14; no longer U320.6 (-), U320.7
- net FOLD_V7: now also U320.6 (-), U320.7; no longer U320.8, U320.9 (-)
- net FOLD_V8: now also U320.8, U320.9 (-); no longer U320.13 (-), U320.14
- net FV6_C: now also U320.12 (+); no longer U320.5 (+)
- net FV7_C: now also U320.5 (+); no longer U320.10 (+)
- net FV8_C: now also U320.10 (+); no longer U320.12 (+)
- net GND: now also C360.1, C415.2, C416.2; no longer C360.2
- net L1V6_C: now also U305.12 (+); no longer U305.5 (+)
- net L1V7_C: now also U305.5 (+); no longer U305.10 (+)
- net L1V8_C: now also U305.10 (+); no longer U305.12 (+)
- net L2V6_C: now also U303.12 (+); no longer U303.5 (+)
- net L2V7_C: now also U303.5 (+); no longer U303.10 (+)
- net L2V8_C: now also U303.10 (+); no longer U303.12 (+)
- net LVL1_V6: now also U305.13 (-), U305.14; no longer U305.6 (-), U305.7
- net LVL1_V7: now also U305.6 (-), U305.7; no longer U305.8, U305.9 (-)
- net LVL1_V8: now also U305.8, U305.9 (-); no longer U305.13 (-), U305.14
- net LVL2_V6: now also U303.13 (-), U303.14; no longer U303.6 (-), U303.7
- net LVL2_V7: now also U303.6 (-), U303.7; no longer U303.13 (-), U303.14
- net P1V5_C: now also U309.3 (+)
- net P1V6_C: now also U309.12 (+)
- net P2V6_C: now also U311.12 (+); no longer U311.5 (+)
- net P2V7_C: now also U311.5 (+); no longer U311.10 (+)
- net P2V8_C: now also U311.10 (+); no longer U311.12 (+)
- net PWM1_V5: now also U309.1, U309.2 (-)
- net PWM1_V6: now also U309.13 (-), U309.14
- net PWM2_V6: now also U311.13 (-), U311.14; no longer U311.6 (-), U311.7
- net PWM2_V7: now also U311.6 (-), U311.7; no longer U311.8, U311.9 (-)
- net PWM2_V8: now also U311.8, U311.9 (-); no longer U311.13 (-), U311.14
- net VCA_V6: now also U319.13 (-), U319.14; no longer U319.6 (-), U319.7
- net VCA_V7: now also U319.6 (-), U319.7; no longer U319.8, U319.9 (-)
- net VCA_V8: now also U319.8, U319.9 (-); no longer U319.13 (-), U319.14
- net P1V7_C: now reaches U314.2 (X6)
- net P1V7_C: now also C416.1, U309.5 (+)
- net P1V8_C: now reaches U314.4 (X7)
- net P1V8_C: now also C415.1, U309.10 (+)
- new net PWM1_V7: U309.6 (-), U309.7
- new net PWM1_V8: U309.8, U309.9 (-)
Other:
- moved on the sheet: C331, C360, U303B, U303C, U303D, U305B, U305C, U305D, U311B, U311C, U311D, U318B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

Commit message: 8V layout rev1
Parts:
- R301, R302: value 12k -> 3k3
Connections:
- net CUTOFF_V7: no longer U318.8, U318.9 (-)
- net LVL2_V7: no longer U303.8, U303.9 (-)
- new net CUTOFF_V8: U318.8, U318.9 (-)
- new net LVL2_V8: U303.8, U303.9 (-)
Changed lines of the file:
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@@
 		)
 	)
-	(global_label "CUTOFF_V7"
+	(global_label "CUTOFF_V8"
 		(shape output)
 		(at 608.33 314.96 0)
@@
 		)
 	)
-	(global_label "LVL2_V7"
+	(global_label "LVL2_V8"
 		(shape output)
 		(at 310.134 399.034 0)
@@
 		(exclude_from_sim no)
 		(in_bom no)
-		(on_board yes)
+		(on_board no)
 		(dnp no)
 		(fields_autoplaced yes)
@@
 			)
 		)
-		(property "Value" "12k"
+		(property "Value" "3k3"
 			(at 30.226 72.136 0)
 			(effects
@@
 		(exclude_from_sim no)
 		(in_bom no)
-		(on_board yes)
+		(on_board no)
 		(dnp no)
 		(fields_autoplaced yes)
@@
 		(exclude_from_sim no)
 		(in_bom no)
-		(on_board yes)
+		(on_board no)
 		(dnp no)
 		(fields_autoplaced yes)
@@
 		(exclude_from_sim no)
 		(in_bom no)
-		(on_board yes)
+		(on_board no)
 		(dnp no)
 		(fields_autoplaced yes)
@@
 		(exclude_from_sim no)
 		(in_bom no)
-		(on_board yes)
+		(on_board no)
 		(dnp no)
 		(fields_autoplaced yes)
@@
 		(exclude_from_sim no)
 		(in_bom no)
-		(on_board yes)
+		(on_board no)
 		(dnp no)
 		(fields_autoplaced yes)
@@
 			)
 		)
-		(property "Value" "12k"
+		(property "Value" "3k3"
 			(at 21.59 72.39 0)
 			(effects
@@
 		(exclude_from_sim no)
 		(in_bom no)
-		(on_board yes)
+		(on_board no)
 		(dnp no)
 		(fields_autoplaced yes)
@@
 		(exclude_from_sim no)
 		(in_bom no)
-		(on_board yes)
+		(on_board no)
 		(dnp no)
 		(fields_autoplaced yes)
@@
 		(exclude_from_sim no)
 		(in_bom no)
-		(on_board yes)
+		(on_board no)
 		(dnp no)
 		(fields_autoplaced yes)
@@
 		(exclude_from_sim no)
 		(in_bom no)
-		(on_board yes)
+		(on_board no)
 		(dnp no)
 		(fields_autoplaced yes)
